File: avionics_board/CAN_Power5.kicad_sch (KiCad schematic)
At the start: 4 parts, among them U17 AP3602AKTR-G1

Commit message: use SAMTEC connectors for AVI to side panels, try HARWIN ones next
Parts:
- renumbered C55 to C54, C56 to C55, C57 to C56, U17 to U16
Changed lines of the file:
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@@
 		(on_board yes)
 		(dnp no)
-		(property "Reference" "C57"
+		(property "Reference" "C56"
 			(at 165.1 104.14 90)
 			(effects
@@
 			(project "AVIONICS_BOARD"
 				(path "/f6cc00ab-17f1-4973-862f-7ac95fe70668/5de22591-2293-4710-b038-9e93720cba0f/c7f59f71-76ca-408f-9d9f-2fe019860d6e"
-					(reference "C57")
+					(reference "C56")
 					(unit 1)
 				)
@@
 		(on_board yes)
 		(dnp no)
-		(property "Reference" "C55"
+		(property "Reference" "C54"
 			(at 121.92 97.79 0)
 			(effects
@@
 			(project "AVIONICS_BOARD"
 				(path "/f6cc00ab-17f1-4973-862f-7ac95fe70668/5de22591-2293-4710-b038-9e93720cba0f/c7f59f71-76ca-408f-9d9f-2fe019860d6e"
-					(reference "C55")
+					(reference "C54")
 					(unit 1)
 				)
@@
 		(dnp no)
 		(fields_autoplaced yes)
-		(property "Reference" "U17"
+		(property "Reference" "U16"
 			(at 154.94 87.63 0)
 			(effects
@@
 			(project "AVIONICS_BOARD"
 				(path "/f6cc00ab-17f1-4973-862f-7ac95fe70668/5de22591-2293-4710-b038-9e93720cba0f/c7f59f71-76ca-408f-9d9f-2fe019860d6e"
-					(reference "U17")
+					(reference "U16")
 					(unit 1)
 				)
@@
 		(dnp no)
 		(fields_autoplaced yes)
-		(property "Reference" "C56"
+		(property "Reference" "C55"
 			(at 177.8 97.7899 0)
 			(effects
@@
 			(project "AVIONICS_BOARD"
 				(path "/f6cc00ab-17f1-4973-862f-7ac95fe70668/5de22591-2293-4710-b038-9e93720cba0f/c7f59f71-76ca-408f-9d9f-2fe019860d6e"
-					(reference "C56")
+					(reference "C55")
 					(unit 1)
 				)
