File: avionics_board/solar_sensor_xy.kicad_sch (KiCad schematic)
At the start: 1 part, among them J13 Conn_02x03_Odd_Even

Commit message: AVI: using through hole M50 connectors for sun detectors and ACS
Parts:
- J12: renamed from J13; footprint Common:SAMTEC-CLP-103-02-X-DH -> Common:HARWIN_M50-3200345; Manufacturer (none) -> Harwin; Part Number (none) -> M50-3200345
Changed lines of the file:
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@@
 		(on_board yes)
 		(dnp no)
-		(property "Reference" "J13"
+		(property "Reference" "J12"
 			(at 143.51 77.47 0)
 			(effects
@@
 			)
 		)
-		(property "Footprint" "Common:SAMTEC-CLP-103-02-X-DH"
+		(property "Footprint" "Common:HARWIN_M50-3200345"
 			(at 144.78 85.725 0)
 			(effects
@@
 			)
 		)
-		(property "Datasheet" "~"
+		(property "Datasheet" "https://cdn.harwin.com/pdfs/M50-320.pdf"
 			(at 144.78 85.725 0)
 			(effects
@@
 			(at 144.78 85.725 0)
 			(effects
+				(font
+					(size 1.27 1.27)
+				)
+				(hide yes)
+			)
+		)
+		(property "Manufacturer" "Harwin"
+			(at 144.78 85.725 0)
+			(effects
+				(font
+					(size 1.27 1.27)
+				)
+				(hide yes)
+			)
+		)
+		(property "Part Number" "M50-3200345"
+			(at 144.78 85.725 0)
+			(effects
