File: avionics_board/solar_sensor_z.kicad_sch (KiCad schematic)
At the start: 1 part, among them J14 Conn_02x05_Odd_Even

Commit message: AVI: using through hole M50 connectors for sun detectors and ACS
Parts:
- J14: footprint Common:SAMTEC_CLP-105-02-X-DH -> Common:HARWIN_M50-3200545; Manufacturer (none) -> Harwin; Part Number (none) -> M50-3200545
Changed lines of the file:
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@@
 			)
 		)
-		(property "Footprint" "Common:SAMTEC_CLP-105-02-X-DH"
+		(property "Footprint" "Common:HARWIN_M50-3200545"
 			(at 144.78 85.725 0)
 			(effects
@@
 			)
 		)
-		(property "Datasheet" "~"
+		(property "Datasheet" "https://cdn.harwin.com/pdfs/M50-320.pdf"
 			(at 144.78 85.725 0)
 			(effects
@@
 			(at 144.78 85.725 0)
 			(effects
+				(font
+					(size 1.27 1.27)
+				)
+				(hide yes)
+			)
+		)
+		(property "Manufacturer" "Harwin"
+			(at 144.78 85.725 0)
+			(effects
+				(font
+					(size 1.27 1.27)
+				)
+				(hide yes)
+			)
+		)
+		(property "Part Number" "M50-3200545"
+			(at 144.78 85.725 0)
+			(effects
