File: avionics_board/CAN_TRANSCEIVER.kicad_sch (KiCad schematic)
At the start: 8 parts, among them U9 TCAN3414

Commit message: clenup BOM for SCI and AUX
Parts:
- C35: Part Number GRM155R61C473KA01D -> GRM155R61H472KA01D; Voltage 16 -> 50
- D6: now fitted
Other:
- note removed: "D = CAN transmit data input, also called TXD, driver input R = CAN receive data output, also called RXD, receiver output"
Changed lines of the file:
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@@
-		)
-	)
-	(text "D = CAN transmit data input, also called TXD, driver input\nR = CAN receive data output, also called RXD, receiver output\n"
-		(exclude_from_sim no)
-		(at 81.28 60.96 0)
-		(effects
-			(font
-				(size 1.27 1.27)
-			)
-			(justify left bottom)
 		)
 	)
@@
 			)
 		)
-		(property "Description" ""
+		(property "Description" "Resistor"
 			(at 165.1 87.63 0)
 			(effects
@@
 			)
 		)
-		(property "Description" ""
+		(property "Description" "Resistor"
 			(at 165.1 95.25 0)
 			(effects
@@
 		(in_bom yes)
 		(on_board yes)
-		(dnp yes)
+		(dnp no)
 		(property "Reference" "D6"
 			(at 193.04 85.725 90)
@@
 			)
 		)
-		(property "Description" ""
+		(property "Description" "TVS DIODE 24VWM 44VC SOT23-3"
 			(at 193.04 91.44 0)
 			(effects
@@
 			)
 		)
-		(property "Description" ""
+		(property "Description" "Unpolarized capacitor"
 			(at 175.26 91.44 0)
 			(effects
@@
 			)
 		)
-		(property "Voltage" "16"
+		(property "Voltage" "50"
 			(at 175.26 97.155 90)
 			(effects
@@
 			)
 		)
-		(property "Part Number" "GRM155R61C473KA01D"
+		(property "Part Number" "GRM155R61H472KA01D"
 			(at 175.26 91.44 0)
 			(effects
@@
 			)
 		)
-		(property "Description" ""
+		(property "Description" "Unpolarized capacitor"
 			(at 105.41 125.73 0)
 			(effects

Commit message: cleaning up bom: remove main camera port since it has not pullups and capacitors, correcting some errors in camera switch
Parts:
- renumbered R42 to R44, R43 to R45
