File: avionics_board/OSC_HSE_TCXO.kicad_sch (KiCad schematic)
At the start: 2 parts, among them X1 10MHz

Commit message: tweaking SCI and AUX for production, using common sheets as much as possible
Parts:
- renumbered C29 to C28
Changed lines of the file:
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@@
 		(on_board yes)
 		(dnp no)
-		(property "Reference" "C29"
+		(property "Reference" "C28"
 			(at 185.801 110.5916 0)
 			(effects
@@
 			(project "aux_board"
 				(path "/85134265-2435-454a-99c4-e49d8e69c5c2/490a0c5b-9225-4953-ad7a-fe6abb29cde0/84780269-b8cb-44bc-ab72-b0ed2668fd84"
-					(reference "C29")
+					(reference "C28")
 					(unit 1)
 				)

Commit message: QC, add second 3V regulator to AUX, INT pullups on AUX SCI AVI
Parts:
- renumbered C28 to C30
Changed lines of the file:
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@@
 		(on_board yes)
 		(dnp no)
-		(property "Reference" "C28"
+		(property "Reference" "C30"
 			(at 185.801 110.5916 0)
 			(effects
@@
 			(project "aux_board"
 				(path "/85134265-2435-454a-99c4-e49d8e69c5c2/490a0c5b-9225-4953-ad7a-fe6abb29cde0/84780269-b8cb-44bc-ab72-b0ed2668fd84"
-					(reference "C28")
+					(reference "C30")
 					(unit 1)
 				)
