File: avionics_board/MAG.kicad_sch (KiCad schematic)
At the start: 8 parts, among them U2 MMC5983MA

Commit message: use SAMTEC connectors for AVI to side panels, try HARWIN ones next
Parts:
- renumbered R17 to R18
Changed lines of the file:
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@@
 		(on_board yes)
 		(dnp no)
-		(property "Reference" "R17"
+		(property "Reference" "R18"
 			(at 110.49 95.25 90)
 			(effects
@@
 			(project "AVIONICS_BOARD"
 				(path "/f6cc00ab-17f1-4973-862f-7ac95fe70668/b4b77cb2-7683-4a8b-8fdc-370cfc88d806"
-					(reference "R17")
+					(reference "R18")
 					(unit 1)
 				)

Commit message: AVI: using through hole M50 connectors for sun detectors and ACS
Parts:
- C21, C22, C23, C24, C25, C26: Order https://www.digikey.com/product-detail/en/samsung-electro-m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 -> (none)
- U2: Order https://www.digikey.com/product-detail/en/memsic-inc/MMC598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 -> (none)
Changed lines of the file:
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@@
-			)
-		)
-		(property "Order" "https://www.digikey.com/product-detail/en/samsung-electro-mechanics/CL10B105KP8NFNC/1276-1945-1-ND/3890031"
-			(at 163.195 73.66 0)
-			(effects
-				(font
-					(size 1.27 1.27)
-				)
-				(hide yes)
 			)
 		)
@@
 			)
 		)
-		(property "Order" "https://www.digikey.com/product-detail/en/samsung-electro-mechanics/CL10X106MO8NRNC/1276-6769-1-ND/5961628"
-			(at 161.29 87.63 0)
-			(effects
-				(font
-					(size 1.27 1.27)
-				)
-				(hide yes)
-			)
-		)
 		(property "Voltage" "25"
 			(at 166.37 90.805 0)
@@
 			)
 		)
-		(property "Order" "https://www.digikey.com/product-detail/en/memsic-inc/MMC5983MA/1267-MMC5983MACT-ND/10452801"
-			(at 137.16 127 0)
-			(effects
-				(font
-					(size 1.27 1.27)
-				)
-				(hide yes)
-			)
-		)
 		(property "Alt" ""
 			(at 140.97 90.17 0)
@@
 			)
 		)
-		(property "Order" "https://www.digikey.com/product-detail/en/samsung-electro-mechanics/CL10X106MO8NRNC/1276-6769-1-ND/5961628"
-			(at 153.67 73.66 0)
-			(effects
-				(font
-					(size 1.27 1.27)
-				)
-				(hide yes)
-			)
-		)
 		(property "Voltage" "25"
 			(at 158.75 76.835 0)
@@
 			)
 		)
-		(property "Order" "https://www.digikey.com/product-detail/en/samsung-electro-mechanics/CL10B105KP8NFNC/1276-1945-1-ND/3890031"
-			(at 163.195 60.325 0)
-			(effects
-				(font
-					(size 1.27 1.27)
-				)
-				(hide yes)
-			)
-		)
 		(property "Voltage" "25"
 			(at 163.195 60.325 0)
@@
 			)
 		)
-		(property "Order" "https://www.digikey.com/product-detail/en/samsung-electro-mechanics/CL10X106MO8NRNC/1276-6769-1-ND/5961628"
-			(at 153.035 87.63 0)
-			(effects
-				(font
-					(size 1.27 1.27)
-				)
-				(hide yes)
-			)
-		)
 		(property "Voltage" "25"
 			(at 158.115 90.805 0)
@@
 			(at 153.67 60.325 0)
 			(effects
-				(font
-					(size 1.27 1.27)
-				)
-				(hide yes)
-			)
-		)
-		(property "Order" "https://www.digikey.com/product-detail/en/samsung-electro-mechanics/CL10X106MO8NRNC/1276-6769-1-ND/5961628"
-			(at 153.67 60.325 0)
-			(effects

Commit message: QC, add second 3V regulator to AUX, INT pullups on AUX SCI AVI
Parts:
- renumbered R18 to R23
Other:
- note removed: "Low ESR cap, close proximity to the chip"
- note removed: "VDD 2.16V to 3.6V Logic 1.62V to 3.6V"
Changed lines of the file:
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@@
-		)
-	)
-	(text "Low ESR cap, close proximity to the chip"
-		(exclude_from_sim no)
-		(at 213.36 86.36 0)
-		(effects
-			(font
-				(size 1.27 1.27)
-			)
-			(justify right bottom)
-		)
-	)
-	(text "VDD 2.16V to 3.6V\n\nLogic 1.62V to 3.6V"
-		(exclude_from_sim no)
-		(at 173.99 105.41 0)
-		(effects
-			(font
-				(size 1.27 1.27)
-			)
-			(justify right bottom)
 		)
 	)
@@
 		(on_board yes)
 		(dnp no)
-		(property "Reference" "R18"
+		(property "Reference" "R23"
 			(at 110.49 95.25 90)
 			(effects
@@
 			(project "AVIONICS_BOARD"
 				(path "/f6cc00ab-17f1-4973-862f-7ac95fe70668/b4b77cb2-7683-4a8b-8fdc-370cfc88d806"
-					(reference "R18")
+					(reference "R23")
 					(unit 1)
 				)

Commit message: AVI board manages its local powers
Parts:
- renumbered R23 to R25
Changed lines of the file:
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@@
 		(on_board yes)
 		(dnp no)
-		(property "Reference" "R23"
+		(property "Reference" "R25"
 			(at 110.49 95.25 90)
 			(effects
@@
 			(project "AVIONICS_BOARD"
 				(path "/f6cc00ab-17f1-4973-862f-7ac95fe70668/b4b77cb2-7683-4a8b-8fdc-370cfc88d806"
-					(reference "R23")
+					(reference "R25")
 					(unit 1)
 				)
