File: avionics_board/MRAM.kicad_sch (KiCad schematic)
At the start: 5 parts, among them U8 MR25H10

Commit message: add SPI CS and MISO pullups and terminations, remove WD from SCI
Parts:
- added R36: 100K, Resistor_SMD:R_0402_1005Metric_Pad0.72x0.64mm_HandSolder, symbol Device:R
Connections:
- net SPI_CS: now also R36.2
- net VDD: now also R36.1
Changed lines of the file:
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@@
+	)
+	(junction
+		(at 120.65 109.22)
+		(diameter 0)
+		(color 0 0 0 0)
 	)
 	(junction
@@
 	)
 	(junction
-		(at 120.65 109.22)
+		(at 111.125 109.22)
+		(diameter 0)
+		(color 0 0 0 0)
+	)
+	(junction
+		(at 111.125 121.92)
 		(diameter 0)
 		(color 0 0 0 0)
@@
 	(wire
 		(pts
+			(xy 111.125 116.84) (xy 111.125 121.92)
+		)
+		(stroke
+			(width 0)
+			(type default)
+		)
+	)
+	(wire
+		(pts
 			(xy 120.65 119.38) (xy 120.65 116.84)
 		)
@@
 	(wire
 		(pts
-			(xy 144.78 121.92) (xy 148.59 121.92)
+			(xy 107.315 121.92) (xy 111.125 121.92)
+		)
+		(stroke
+			(width 0)
+			(type default)
+		)
+	)
+	(wire
+		(pts
+			(xy 111.125 109.22) (xy 120.65 109.22)
+		)
+		(stroke
+			(width 0)
+			(type default)
+		)
+	)
+	(wire
+		(pts
+			(xy 130.81 109.22) (xy 158.75 109.22)
+		)
+		(stroke
+			(width 0)
+			(type default)
+		)
+	)
+	(wire
+		(pts
+			(xy 198.12 115.57) (xy 198.12 109.22)
+		)
+		(stroke
+			(width 0)
+			(type default)
+		)
+	)
+	(wire
+		(pts
+			(xy 158.75 130.81) (xy 158.75 137.16)
+		)
+		(stroke
+			(width 0)
+			(type default)
+		)
+	)
+	(wire
+		(pts
+			(xy 120.65 119.38) (xy 148.59 119.38)
+		)
+		(stroke
+			(width 0)
+			(type default)
+		)
+	)
+	(wire
+		(pts
+			(xy 111.125 121.92) (xy 148.59 121.92)
 		)
 		(stroke
@@
 	(wire
 		(pts
-			(xy 130.81 109.22) (xy 158.75 109.22)
-		)
-		(stroke
-			(width 0)
-			(type default)
-		)
-	)
-	(wire
-		(pts
-			(xy 198.12 115.57) (xy 198.12 109.22)
-		)
-		(stroke
-			(width 0)
-			(type default)
-		)
-	)
-	(wire
-		(pts
-			(xy 158.75 130.81) (xy 158.75 137.16)
-		)
-		(stroke
-			(width 0)
-			(type default)
-		)
-	)
-	(wire
-		(pts
-			(xy 120.65 119.38) (xy 148.59 119.38)
-		)
-		(stroke
-			(width 0)
-			(type default)
-		)
-	)
-	(wire
-		(pts
 			(xy 158.75 137.16) (xy 198.12 137.16)
 		)
@@
 	(wire
 		(pts
-			(xy 120.65 103.505) (xy 120.65 109.22)
+			(xy 111.125 103.505) (xy 111.125 109.22)
 		)
 		(stroke
@@
 	(hierarchical_label "VDD"
 		(shape output)
-		(at 120.65 103.505 180)
+		(at 111.125 103.505 180)
 		(fields_autoplaced yes)
 		(effects
@@
 	(hierarchical_label "SPI_CS"
 		(shape output)
-		(at 144.78 121.92 180)
+		(at 107.315 121.92 180)
 		(fields_autoplaced yes)
 		(effects
@@
 			(project ""
 				(path "/b4b2c88d-f6cd-4e60-862d-e21f68728580/f3d5c282-94c3-4259-817b-bad3ee4bc8e5"
-					(reference "C59")
+					(reference "C58")
 					(unit 1)
 				)
@@
 			(project ""
 				(path "/b4b2c88d-f6cd-4e60-862d-e21f68728580/f3d5c282-94c3-4259-817b-bad3ee4bc8e5"
-					(reference "U26")
+					(reference "U25")
 					(unit 1)
 				)
@@
 			(project ""
 				(path "/b4b2c88d-f6cd-4e60-862d-e21f68728580/f3d5c282-94c3-4259-817b-bad3ee4bc8e5"
-					(reference "R38")
+					(reference "R37")
 					(unit 1)
 				)
@@
 			(project ""
 				(path "/f6cc00ab-17f1-4973-862f-7ac95fe70668/00000000-0000-0000-0000-00005ea31c93/00000000-0000-0000-0000-00006310c53d"
-					(reference "R30")
+					(reference "R31")
 					(unit 1)
 				)
@@
 			(project ""
 				(path "/b4b2c88d-f6cd-4e60-862d-e21f68728580/f3d5c282-94c3-4259-817b-bad3ee4bc8e5"
-					(reference "R39")
+					(reference "R38")
 					(unit 1)
 				)
@@
 			(project ""
 				(path "/f6cc00ab-17f1-4973-862f-7ac95fe70668/00000000-0000-0000-0000-00005ea31c93/00000000-0000-0000-0000-00006310c53d"
-					(reference "R31")
+					(reference "R32")
+					(unit 1)
+				)
+			)
+		)
+	)
+	(symbol
+		(lib_id "Device:R")
+		(at 111.125 113.03 0)
+		(unit 1)
+		(exclude_from_sim no)
+		(in_bom yes)
+		(on_board yes)
+		(dnp no)
+		(property "Reference" "R36"
+			(at 113.665 111.76 0)
+			(effects
+				(font
+					(size 1.27 1.27)
+				)
+				(justify left)
+			)
+		)
+		(property "Value" "100K"
+			(at 112.903 114.173 0)
+			(effects
+				(font
+					(size 1.27 1.27)
+				)
+				(justify left)
+			)
+		)
+		(property "Footprint" "Resistor_SMD:R_0402_1005Metric_Pad0.72x0.64mm_HandSolder"
+			(at 109.347 113.03 90)
+			(effects
+				(font
+					(size 1.27 1.27)
+				)
+				(hide yes)
+			)
+		)
+		(property "Datasheet" "https://www.yageo.com/upload/media/product/products/datasheet/rchip/PYu-RC_Group_51_RoHS_L_12.pdf"
+			(at 111.125 113.03 0)
+			(effects
+				(font
+					(size 1.27 1.27)
+				)
+				(hide yes)
+			)
+		)
+		(property "Description" ""
+			(at 111.125 113.03 0)
+			(effects
+				(font
+					(size 1.27 1.27)
+				)
+				(hide yes)
+			)
+		)
+		(property "Alt" ""
+			(at 111.125 113.03 0)
+			(effects
+				(font
+					(size 1.27 1.27)
+				)
+				(hide yes)
+			)
+		)
+		(property "Manufacturer" "YAGEO"
+			(at 111.125 113.03 0)
+			(effects
+				(font
+					(size 1.27 1.27)
+				)
+				(hide yes)
+			)
+		)
+		(property "Note" "generic pullup/down"
+			(at 111.125 113.03 0)
+			(effects
+				(font
+					(size 1.27 1.27)
+				)
+				(hide yes)
+			)
+		)
+		(property "Part Number" "RC0402FR-07100KL"
+			(at 111.125 113.03 0)
+			(effects
+				(font
+					(size 1.27 1.27)
+				)
+				(hide yes)
+			)
+		)
+		(property "Tolerance" "1"
+			(at 111.125 113.03 0)
+			(effects
+				(font
+					(size 1.27 1.27)
+				)
+				(hide yes)
+			)
+		)
+		(pin "1"
+		)
+		(pin "2"
+		)
+		(instances
+			(project "sci_board"
+				(path "/b4b2c88d-f6cd-4e60-862d-e21f68728580/f3d5c282-94c3-4259-817b-bad3ee4bc8e5"
+					(reference "R36")
+					(unit 1)
+				)
+			)
+			(project "AVIONICS_BOARD"
+				(path "/f6cc00ab-17f1-4973-862f-7ac95fe70668/00000000-0000-0000-0000-00005ea31c93/00000000-0000-0000-0000-00006310c53d"
+					(reference "R30")
 					(unit 1)
 				)
@@
 			(project "sci_board"
 				(path "/b4b2c88d-f6cd-4e60-862d-e21f68728580/f3d5c282-94c3-4259-817b-bad3ee4bc8e5"
-					(reference "R40")
+					(reference "R39")
 					(unit 1)
 				)
@@
 			(project ""
 				(path "/f6cc00ab-17f1-4973-862f-7ac95fe70668/00000000-0000-0000-0000-00005ea31c93/00000000-0000-0000-0000-00006310c53d"
-					(reference "R32")
-					(unit 1)
-				)
+					(reference "R33")
+					(unit 1)
+				)

Commit message: cleaning up bom: remove main camera port since it has not pullups and capacitors, correcting some errors in camera switch
Parts:
- renumbered C33 to C30, R36 to R39, R39 to R40, R40 to R41, R162 to R42, U8 to U7
