File: avionics_board/acs_directional_unit.kicad_sch (KiCad schematic)
At the start: 7 parts, among them J8 Conn_01x04, U13 INA226, U14 DRV8838

Commit message: add headers for ACS and sun sensors
Parts:
- removed J8: Conn_01x04, Connector_PinHeader_2.54mm:PinHeader_1x04_P2.54mm_Vertical, symbol Connector:Conn_01x04_Pin
Connections:
- net OUT_P: now reaches U14.2 (OUT1)
- net OUT_N: now reaches U14.3 (OUT2)
Changed lines of the file:
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@@
 	(wire
 		(pts
-			(xy 181.61 113.03) (xy 181.61 109.22)
+			(xy 133.35 83.82) (xy 137.16 83.82)
 		)
 		(stroke
@@
 		)
 	)
+	(polyline
+		(pts
+			(xy 243.84 59.69) (xy 243.84 80.01)
+		)
+		(stroke
+			(width 0)
+			(type dash)
+		)
+	)
+	(polyline
+		(pts
+			(xy 205.74 66.04) (xy 257.81 66.04)
+		)
+		(stroke
+			(width 0)
+			(type dash)
+		)
+	)
 	(wire
 		(pts
-			(xy 191.77 104.14) (xy 191.77 106.68)
+			(xy 146.685 97.79) (xy 146.685 97.155)
 		)
 		(stroke
@@
 	(wire
 		(pts
-			(xy 133.35 83.82) (xy 137.16 83.82)
+			(xy 149.86 107.95) (xy 142.24 107.95)
 		)
 		(stroke
@@
 	(wire
 		(pts
-			(xy 181.61 101.6) (xy 191.77 101.6)
+			(xy 137.16 83.82) (xy 137.16 83.185)
 		)
 		(stroke
@@
 	(polyline
 		(pts
-			(xy 243.84 59.69) (xy 243.84 80.01)
+			(xy 205.74 76.2) (xy 257.81 76.2)
 		)
 		(stroke
@@
 	(wire
 		(pts
-			(xy 181.61 109.22) (xy 191.77 109.22)
+			(xy 142.24 105.41) (xy 149.86 105.41)
 		)
 		(stroke
@@
 	(polyline
 		(pts
-			(xy 205.74 66.04) (xy 257.81 66.04)
+			(xy 219.71 59.69) (xy 219.71 80.01)
 		)
 		(stroke
@@
 	(wire
 		(pts
-			(xy 146.685 97.79) (xy 146.685 97.155)
+			(xy 137.16 77.47) (xy 133.35 77.47)
 		)
 		(stroke
@@
 	(wire
 		(pts
-			(xy 149.86 107.95) (xy 142.24 107.95)
+			(xy 146.685 92.075) (xy 146.685 91.44)
 		)
 		(stroke
@@
 	(wire
 		(pts
-			(xy 137.16 83.82) (xy 137.16 83.185)
+			(xy 126.365 62.865) (xy 126.365 62.23)
 		)
 		(stroke
@@
 		)
 	)
+	(wire
+		(pts
+			(xy 142.24 102.87) (xy 149.86 102.87)
+		)
+		(stroke
+			(width 0)
+			(type default)
+		)
+	)
+	(wire
+		(pts
+			(xy 145.415 83.82) (xy 160.02 83.82)
+		)
+		(stroke
+			(width 0)
+			(type default)
+		)
+	)
+	(wire
+		(pts
+			(xy 137.16 77.47) (xy 137.16 78.105)
+		)
+		(stroke
+			(width 0)
+			(type default)
+		)
+	)
+	(wire
+		(pts
+			(xy 137.16 83.82) (xy 145.415 83.82)
+		)
+		(stroke
+			(width 0)
+			(type default)
+		)
+	)
+	(wire
+		(pts
+			(xy 157.48 91.44) (xy 157.48 92.71)
+		)
+		(stroke
+			(width 0)
+			(type default)
+		)
+	)
 	(polyline
 		(pts
-			(xy 205.74 76.2) (xy 257.81 76.2)
+			(xy 205.74 71.12) (xy 257.81 71.12)
 		)
 		(stroke
@@
 		)
 	)
+	(polyline
+		(pts
+			(xy 226.06 59.69) (xy 226.06 80.01)
+		)
+		(stroke
+			(width 0)
+			(type dash)
+		)
+	)
 	(wire
 		(pts
-			(xy 142.24 105.41) (xy 149.86 105.41)
+			(xy 123.19 56.515) (xy 123.19 62.23)
 		)
 		(stroke
@@
 		)
 	)
+	(wire
+		(pts
+			(xy 126.365 57.15) (xy 126.365 56.515)
+		)
+		(stroke
+			(width 0)
+			(type default)
+		)
+	)
+	(wire
+		(pts
+			(xy 160.02 120.015) (xy 160.02 118.11)
+		)
+		(stroke
+			(width 0)
+			(type default)
+		)
+	)
 	(polyline
 		(pts
-			(xy 219.71 59.69) (xy 219.71 80.01)
+			(xy 213.36 59.69) (xy 213.36 80.01)
 		)
 		(stroke
@@
 		)
 	)
-	(wire
-		(pts
-			(xy 137.16 77.47) (xy 133.35 77.47)
-		)
-		(stroke
-			(width 0)
-			(type default)
-		)
-	)
-	(wire
-		(pts
-			(xy 146.685 92.075) (xy 146.685 91.44)
-		)
-		(stroke
-			(width 0)
-			(type default)
-		)
-	)
-	(wire
-		(pts
-			(xy 126.365 62.865) (xy 126.365 62.23)
-		)
-		(stroke
-			(width 0)
-			(type default)
-		)
-	)
-	(wire
-		(pts
-			(xy 142.24 102.87) (xy 149.86 102.87)
-		)
-		(stroke
-			(width 0)
-			(type default)
-		)
-	)
-	(wire
-		(pts
-			(xy 145.415 83.82) (xy 160.02 83.82)
-		)
-		(stroke
-			(width 0)
-			(type default)
-		)
-	)
-	(wire
-		(pts
-			(xy 137.16 77.47) (xy 137.16 78.105)
-		)
-		(stroke
-			(width 0)
-			(type default)
-		)
-	)
-	(wire
-		(pts
-			(xy 137.16 83.82) (xy 145.415 83.82)
-		)
-		(stroke
-			(width 0)
-			(type default)
-		)
-	)
-	(wire
-		(pts
-			(xy 181.61 97.79) (xy 181.61 101.6)
-		)
-		(stroke
-			(width 0)
-			(type default)
-		)
-	)
-	(wire
-		(pts
-			(xy 157.48 91.44) (xy 157.48 92.71)
-		)
-		(stroke
-			(width 0)
-			(type default)
-		)
-	)
 	(polyline
 		(pts
-			(xy 205.74 71.12) (xy 257.81 71.12)
+			(xy 256.54 59.69) (xy 256.54 80.01)
 		)
 		(stroke
@@
 		)
 	)
-	(polyline
-		(pts
-			(xy 226.06 59.69) (xy 226.06 80.01)
-		)
-		(stroke
-			(width 0)
-			(type dash)
-		)
-	)
-	(wire
-		(pts
-			(xy 123.19 56.515) (xy 123.19 62.23)
-		)
-		(stroke
-			(width 0)
-			(type default)
-		)
-	)
-	(wire
-		(pts
-			(xy 126.365 57.15) (xy 126.365 56.515)
-		)
-		(stroke
-			(width 0)
-			(type default)
-		)
-	)
-	(wire
-		(pts
-			(xy 160.02 120.015) (xy 160.02 118.11)
-		)
-		(stroke
-			(width 0)
-			(type default)
-		)
-	)
-	(polyline
-		(pts
-			(xy 213.36 59.69) (xy 213.36 80.01)
-		)
-		(stroke
-			(width 0)
-			(type dash)
-		)
-	)
-	(polyline
-		(pts
-			(xy 256.54 59.69) (xy 256.54 80.01)
-		)
-		(stroke
-			(width 0)
-			(type dash)
-		)
-	)
 	(text "L"
 		(exclude_from_sim no)
@@
 		)
 	)
+	(hierarchical_label "OUT_P"
+		(shape output)
+		(at 181.61 97.79 0)
+		(fields_autoplaced yes)
+		(effects
+			(font
+				(size 1.27 1.27)
+			)
+			(justify left)
+		)
+	)
 	(hierarchical_label "PWR_LOGIC"
 		(shape input)
@@
 		(shape input)
 		(at 145.415 88.9 0)
+		(fields_autoplaced yes)
+		(effects
+			(font
+				(size 1.27 1.27)
+			)
+			(justify left)
+		)
+	)
+	(hierarchical_label "OUT_N"
+		(shape output)
+		(at 181.61 113.03 0)
 		(fields_autoplaced yes)
 		(effects
@@
 					(unit 1)
 				)
-			)
-		)
-	)
-	(symbol
-		(lib_id "Connector:Conn_01x04_Pin")
-		(at 196.85 106.68 180)
-		(unit 1)
-		(exclude_from_sim no)
-		(in_bom yes)
-		(on_board yes)
-		(dnp yes)
-		(property "Reference" "J8"
-			(at 196.85 96.52 0)
-			(effects
-				(font
-					(size 1.27 1.27)
-				)
-			)
-		)
-		(property "Value" "Conn_01x04"
-			(at 198.12 99.06 0)
-			(effects
-				(font
-					(size 1.27 1.27)
-				)
-			)
-		)
-		(property "Footprint" "Connector_PinHeader_2.54mm:PinHeader_1x04_P2.54mm_Vertical"
-			(at 196.85 106.68 0)
-			(effects
-				(font
-					(size 1.27 1.27)
-				)
-				(hide yes)
-			)
-		)
-		(property "Datasheet" "~"
-			(at 196.85 106.68 0)
-			(effects
-				(font
-					(size 1.27 1.27)
-				)
-				(hide yes)
-			)
-		)
-		(property "Description" "Generic connector, single row, 01x04, script generated"
-			(at 196.85 106.68 0)
-			(effects
-				(font
-					(size 1.27 1.27)
-				)
-				(hide yes)
-			)
-		)
-		(property "Alt" ""
-			(at 196.85 106.68 0)
-			(effects
-				(font
-					(size 1.27 1.27)
-				)
-				(hide yes)
-			)
-		)
-		(pin "1"
-		)
-		(pin "2"
-		)
-		(pin "4"
-		)
-		(pin "3"
-		)
-		(instances
-			(project "AVIONICS_BOARD"
-				(path "/f6cc00ab-17f1-4973-862f-7ac95fe70668/1f9ae17d-3f3e-4633-9b01-30c344473415/4e2a47c2-c2ed-4db2-bf85-7030d7458163"
-					(reference "J8")
-					(unit 1)
-				)
-				(path "/f6cc00ab-17f1-4973-862f-7ac95fe70668/1f9ae17d-3f3e-4633-9b01-30c344473415/7d3e76d7-4668-440d-8487-c4215eabf8a2"
-					(reference "J4")
-					(unit 1)
-				)
-				(path "/f6cc00ab-17f1-4973-862f-7ac95fe70668/1f9ae17d-3f3e-4633-9b01-30c344473415/a0859814-3829-45a9-a25d-0db563664eca"
-					(reference "J1")
-					(unit 1)
-				)

Commit message: use SAMTEC connectors for AVI to side panels, try HARWIN ones next
Parts:
- renumbered R40 to R41
Changed lines of the file:
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@@
 		(on_board yes)
 		(dnp no)
-		(property "Reference" "R40"
+		(property "Reference" "R41"
 			(at 139.065 79.3749 0)
 			(effects
@@
 			(project "AVIONICS_BOARD"
 				(path "/f6cc00ab-17f1-4973-862f-7ac95fe70668/1f9ae17d-3f3e-4633-9b01-30c344473415/4e2a47c2-c2ed-4db2-bf85-7030d7458163"
-					(reference "R40")
+					(reference "R41")
 					(unit 1)
 				)
 				(path "/f6cc00ab-17f1-4973-862f-7ac95fe70668/1f9ae17d-3f3e-4633-9b01-30c344473415/7d3e76d7-4668-440d-8487-c4215eabf8a2"
-					(reference "R28")
+					(reference "R29")
 					(unit 1)
 				)
 				(path "/f6cc00ab-17f1-4973-862f-7ac95fe70668/1f9ae17d-3f3e-4633-9b01-30c344473415/a0859814-3829-45a9-a25d-0db563664eca"
-					(reference "R20")
+					(reference "R21")
 					(unit 1)
 				)

Commit message: AVI: using through hole M50 connectors for sun detectors and ACS
Parts:
- U14: Order https://www.digikey.com/product-detail/en/texas-instruments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 -> (none)
Changed lines of the file:
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@@
-			)
-		)
-		(property "Order" "https://www.digikey.com/product-detail/en/texas-instruments/DRV8838DSGR/296-40081-1-ND/5177958"
-			(at 160.02 105.41 0)
-			(effects
-				(font
-					(size 1.27 1.27)
-				)
-				(hide yes)
 			)
 		)

Commit message: add SPI CS and MISO pullups and terminations, remove WD from SCI
Parts:
- renumbered R41 to R42
Changed lines of the file:
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@@
 		(on_board yes)
 		(dnp no)
-		(property "Reference" "R41"
+		(property "Reference" "R42"
 			(at 139.065 79.3749 0)
 			(effects
@@
 			(project "AVIONICS_BOARD"
 				(path "/f6cc00ab-17f1-4973-862f-7ac95fe70668/1f9ae17d-3f3e-4633-9b01-30c344473415/4e2a47c2-c2ed-4db2-bf85-7030d7458163"
-					(reference "R41")
+					(reference "R42")
 					(unit 1)
 				)

Commit message: QC, add second 3V regulator to AUX, INT pullups on AUX SCI AVI
Parts:
- renumbered R42 to R46
Changed lines of the file:
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@@
 		(on_board yes)
 		(dnp no)
-		(property "Reference" "R42"
+		(property "Reference" "R46"
 			(at 139.065 79.3749 0)
 			(effects
@@
 			(project "AVIONICS_BOARD"
 				(path "/f6cc00ab-17f1-4973-862f-7ac95fe70668/1f9ae17d-3f3e-4633-9b01-30c344473415/4e2a47c2-c2ed-4db2-bf85-7030d7458163"
-					(reference "R42")
+					(reference "R46")
 					(unit 1)
 				)
 				(path "/f6cc00ab-17f1-4973-862f-7ac95fe70668/1f9ae17d-3f3e-4633-9b01-30c344473415/7d3e76d7-4668-440d-8487-c4215eabf8a2"
-					(reference "R29")
+					(reference "R33")
 					(unit 1)
 				)
 				(path "/f6cc00ab-17f1-4973-862f-7ac95fe70668/1f9ae17d-3f3e-4633-9b01-30c344473415/a0859814-3829-45a9-a25d-0db563664eca"
-					(reference "R21")
+					(reference "R25")
 					(unit 1)
 				)

Commit message: AVI board manages its local powers
Parts:
- renumbered R46 to R48
Changed lines of the file:
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@@
 		(on_board yes)
 		(dnp no)
-		(property "Reference" "R46"
+		(property "Reference" "R48"
 			(at 139.065 79.3749 0)
 			(effects
@@
 			(project "AVIONICS_BOARD"
 				(path "/f6cc00ab-17f1-4973-862f-7ac95fe70668/1f9ae17d-3f3e-4633-9b01-30c344473415/4e2a47c2-c2ed-4db2-bf85-7030d7458163"
-					(reference "R46")
+					(reference "R48")
 					(unit 1)
 				)
 				(path "/f6cc00ab-17f1-4973-862f-7ac95fe70668/1f9ae17d-3f3e-4633-9b01-30c344473415/7d3e76d7-4668-440d-8487-c4215eabf8a2"
-					(reference "R33")
+					(reference "R35")
 					(unit 1)
 				)
 				(path "/f6cc00ab-17f1-4973-862f-7ac95fe70668/1f9ae17d-3f3e-4633-9b01-30c344473415/a0859814-3829-45a9-a25d-0db563664eca"
-					(reference "R25")
+					(reference "R27")
 					(unit 1)
 				)
