File: eps_board/BATTERY.kicad_sch (KiCad schematic)
At the start: 15 parts, among them J9 Conn_01x02_Female, U16 MIC2009YM6-TR

Commit message: EPS use M50 2x3 connectors for solar cells. remove 2 connectors since they are all tied together and top/bottom can be routed through sides and side connectors
Parts:
- J9: value Conn_01x02_Female -> Conn_01x02
Changed lines of the file:
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@@
 			)
 		)
-		(property "Value" "Conn_01x02_Female"
+		(property "Value" "Conn_01x02"
 			(at 215.9762 54.229 0)
 			(effects

Commit message: cleaning up bom: remove main camera port since it has not pullups and capacitors, correcting some errors in camera switch
Parts:
- R69: renamed from R67; value 3.09K -> 988R; footprint Resistor_SMD:R_0402_1005Metric_Pad0.72x0.64mm_HandSolder -> Resistor_SMD:R_0603_1608Metric_Pad0.98x0.95mm_HandSolder; Part Number RC0402FR-073K09L -> RT0603DRE07988RL; Tolerance 1 -> 0.5
- U15: renamed from U16; value MIC2009YM6-TR -> MIC2009A-1YM6-TR; Part Number MIC2009YM6-TR -> MIC2009A-1YM6-TR
- renumbered C61 to C56, C62 to C57, C63 to C58, J9 to J7, R64 to R66, R65 to R67, R66 to R68, R68 to R70, R69 to R71
Other:
- note added: "200mA"
- note removed: "150mA current Limit set by 3090 Ohm resistor"
