File: eps_board/BATTERY_CHARGER.kicad_sch (KiCad schematic)
At the start: 14 parts, among them U14 LTC4066

Commit message: cleaning up bom: remove main camera port since it has not pullups and capacitors, correcting some errors in camera switch
Parts:
- renumbered C53 to C48, C54 to C49, C55 to C50, C56 to C51, R48 to R50, R49 to R51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
