File: eps_board/IDEAL_DIODE.kicad_sch (KiCad schematic)
At the start: 7 parts, among them U20 TPS2115ADRBR

Commit message: cleaning up bom: remove main camera port since it has not pullups and capacitors, correcting some errors in camera switch
Parts:
- R81: renamed from R79; value 330 -> 330R
- renumbered C67 to C62, C68 to C63, R76 to R78, R77 to R79, R78 to R80, U20 to U19
