File: eps_board/PMIC.kicad_sch (KiCad schematic)
At the start: 32 parts, among them U5 STM32L496ZGTx

Commit message: cleaning up bom: remove main camera port since it has not pullups and capacitors, correcting some errors in camera switch
Parts:
- C18: renamed from C21; value 1uF -> 10uF; Part Number GRM188R61C105KA12D -> GRM188R61E106KA73D
- C25: renamed from C28; value 1uF -> 10uF; Part Number GRM188R61C105KA12D -> GRM188R61E106KA73D
- C8: renamed from C10; value 1uF -> 10uF; Part Number GRM188R61C105KA12D -> GRM188R61E106KA73D
- renumbered C12 to C10, C13 to C11, C14 to C12, C16 to C13, C17 to C14, C18 to C15, C19 to C16, C20 to C17, C22 to C19, C23 to C20, C24 to C21, C25 to C22, C26 to C23, C27 to C24, C11 to C9, U5 to U4
