File: eps_board/power_selector.kicad_sch (KiCad schematic)
At the start: 16 parts, among them U43 LM66200DRLR, U44 LM66200DRLR

Commit message: cleaning up bom: remove main camera port since it has not pullups and capacitors, correcting some errors in camera switch
Parts:
- renumbered C101 to C96, C102 to C97, R115 to R117, R116 to R118, R117 to R119, R118 to R120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
