File: eps_board/CURRENT_MONITOR.kicad_sch (KiCad schematic)
At the start: 7 parts, among them U1 MIC2009YM6-TR, U2 INA226AIDGSR

Commit message: cleaning up bom: remove main camera port since it has not pullups and capacitors, correcting some errors in camera switch
Parts:
- C75: renamed from C2; value 1uF -> 10uF; Part Number GRM188R61C105KA12D -> GRM188R61E106KA73D
- U27: renamed from U1; value MIC2009YM6-TR -> MIC2009A-1YM6-TR; Part Number MIC2009YM6-TR -> MIC2009A-1YM6-TR
- renumbered C1 to C74, C3 to C76, R19 to R95, R20 to R96, U2 to U28

Commit message: propate the changes to RF
Parts:
- renumbered C74 to C1, C75 to C2, C76 to C3, R95 to R19, R96 to R20, U27 to U1, U28 to U2

Commit message: tweaks before merge
Parts:
- renumbered C1 to C74, C2 to C75, C3 to C76, R19 to R95, R20 to R96, U1 to U27, U2 to U28
Changed lines of the file:
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@@
 		(dnp no)
 		(fields_autoplaced yes)
-		(property "Reference" "C3"
+		(property "Reference" "C76"
 			(at 111.125 93.9799 0)
 			(effects
@@
 		(dnp no)
 		(fields_autoplaced yes)
-		(property "Reference" "U2"
+		(property "Reference" "U28"
 			(at 132.08 48.26 0)
 			(effects
@@
 		(on_board yes)
 		(dnp no)
-		(property "Reference" "R20"
+		(property "Reference" "R96"
 			(at 109.22 71.12 0)
 			(effects
@@
 		(dnp no)
 		(fields_autoplaced yes)
-		(property "Reference" "C1"
+		(property "Reference" "C74"
 			(at 160.655 58.4199 0)
 			(effects
@@
 		(dnp no)
 		(fields_autoplaced yes)
-		(property "Reference" "U1"
+		(property "Reference" "U27"
 			(at 69.215 60.96 0)
 			(effects
@@
 		(on_board yes)
 		(dnp no)
-		(property "Reference" "C2"
+		(property "Reference" "C75"
 			(at 96.52 64.77 0)
 			(effects
@@
 		(on_board yes)
 		(dnp no)
-		(property "Reference" "R19"
+		(property "Reference" "R95"
 			(at 168.91 58.42 0)
 			(effects

Commit message: local switches and monitors for SCI and RF
Parts:
- renumbered C74 to C52, C75 to C53, C76 to C54, R95 to R33, R96 to R34, U27 to U13, U28 to U14
