File: sci_board/camera.kicad_sch (KiCad schematic)
At the start: 11 parts, among them J2 10051922-2410EHLF

Commit message: tweaking SCI and AUX for production, using common sheets as much as possible
Parts:
- renumbered J2 to J3, R12 to R14, R13 to R15
Changed lines of the file:
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@@
 		(on_board yes)
 		(dnp no)
-		(property "Reference" "J2"
+		(property "Reference" "J3"
 			(at 136.525 106.045 0)
 			(effects
@@
 			(project "sci_board"
 				(path "/b4b2c88d-f6cd-4e60-862d-e21f68728580/5e5b27f8-7a4c-45d0-95f8-aff71797fcd3/21d0e59e-a5df-4633-9634-c7d789255f22"
-					(reference "J2")
+					(reference "J3")
 					(unit 1)
 				)
 				(path "/b4b2c88d-f6cd-4e60-862d-e21f68728580/5e5b27f8-7a4c-45d0-95f8-aff71797fcd3/3e22df28-91f0-4c0f-b958-7bfd7fe99c70"
-					(reference "J3")
+					(reference "J4")
 					(unit 1)
 				)
 				(path "/b4b2c88d-f6cd-4e60-862d-e21f68728580/5e5b27f8-7a4c-45d0-95f8-aff71797fcd3/87e2c931-24b0-464d-a54c-5e253d37e662"
-					(reference "J4")
+					(reference "J5")
 					(unit 1)
 				)
@@
 		(dnp no)
 		(fields_autoplaced yes)
-		(property "Reference" "R12"
+		(property "Reference" "R14"
 			(at 45.72 64.1349 0)
 			(effects
@@
 			(project "sci_board"
 				(path "/b4b2c88d-f6cd-4e60-862d-e21f68728580/5e5b27f8-7a4c-45d0-95f8-aff71797fcd3/21d0e59e-a5df-4633-9634-c7d789255f22"
-					(reference "R12")
+					(reference "R14")
 					(unit 1)
 				)
 				(path "/b4b2c88d-f6cd-4e60-862d-e21f68728580/5e5b27f8-7a4c-45d0-95f8-aff71797fcd3/3e22df28-91f0-4c0f-b958-7bfd7fe99c70"
-					(reference "R14")
+					(reference "R16")
 					(unit 1)
 				)
 				(path "/b4b2c88d-f6cd-4e60-862d-e21f68728580/5e5b27f8-7a4c-45d0-95f8-aff71797fcd3/87e2c931-24b0-464d-a54c-5e253d37e662"
-					(reference "R16")
+					(reference "R18")
 					(unit 1)
 				)
@@
 		(dnp no)
 		(fields_autoplaced yes)
-		(property "Reference" "R13"
+		(property "Reference" "R15"
 			(at 62.23 64.1349 0)
 			(effects
@@
 			(project "sci_board"
 				(path "/b4b2c88d-f6cd-4e60-862d-e21f68728580/5e5b27f8-7a4c-45d0-95f8-aff71797fcd3/21d0e59e-a5df-4633-9634-c7d789255f22"
-					(reference "R13")
+					(reference "R15")
 					(unit 1)
 				)
 				(path "/b4b2c88d-f6cd-4e60-862d-e21f68728580/5e5b27f8-7a4c-45d0-95f8-aff71797fcd3/3e22df28-91f0-4c0f-b958-7bfd7fe99c70"
-					(reference "R15")
+					(reference "R17")
 					(unit 1)
 				)
 				(path "/b4b2c88d-f6cd-4e60-862d-e21f68728580/5e5b27f8-7a4c-45d0-95f8-aff71797fcd3/87e2c931-24b0-464d-a54c-5e253d37e662"
-					(reference "R17")
-					(unit 1)
-				)
+					(reference "R19")
+					(unit 1)
+				)

Commit message: clenup BOM for SCI and AUX
Parts:
- J3: Manufacturer (none) -> Amphenol; Part Number (none) -> 10051922-2410EHLF
Changed lines of the file:
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@@
+			)
+		)
+		(property "Part Number" "10051922-2410EHLF"
+			(at 149.225 99.06 0)
+			(effects
+				(font
+					(size 1.27 1.27)
+				)
+				(hide yes)
+			)
+		)
+		(property "Manufacturer" "Amphenol"
+			(at 149.225 99.06 0)
+			(effects
+				(font
+					(size 1.27 1.27)
+				)
+				(hide yes)
 			)
 		)

Commit message: cleaning up bom: remove main camera port since it has not pullups and capacitors, correcting some errors in camera switch
Parts:
- added R17, R20: 10K, Resistor_SMD:R_0402_1005Metric_Pad0.72x0.64mm_HandSolder, symbol Device:R
Connections:
- net 3V3: now also R17.1, R20.1
- net SCK: now also R20.2
- net SDA: now also R17.2

Commit message: QC, add second 3V regulator to AUX, INT pullups on AUX SCI AVI
Parts:
- renumbered R14 to R17, R15 to R18, R20 to R19, R17 to R20
Changed lines of the file:
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@@
 		(dnp no)
 		(fields_autoplaced yes)
-		(property "Reference" "R17"
+		(property "Reference" "R20"
 			(at 59.055 89.5349 0)
 			(effects
@@
 			(project "sci_board"
 				(path "/b4b2c88d-f6cd-4e60-862d-e21f68728580/5e5b27f8-7a4c-45d0-95f8-aff71797fcd3/21d0e59e-a5df-4633-9634-c7d789255f22"
-					(reference "R17")
+					(reference "R20")
 					(unit 1)
 				)
 				(path "/b4b2c88d-f6cd-4e60-862d-e21f68728580/5e5b27f8-7a4c-45d0-95f8-aff71797fcd3/3e22df28-91f0-4c0f-b958-7bfd7fe99c70"
-					(reference "R21")
+					(reference "R24")
 					(unit 1)
 				)
 				(path "/b4b2c88d-f6cd-4e60-862d-e21f68728580/5e5b27f8-7a4c-45d0-95f8-aff71797fcd3/87e2c931-24b0-464d-a54c-5e253d37e662"
-					(reference "R25")
+					(reference "R28")
 					(unit 1)
 				)
@@
 		(dnp no)
 		(fields_autoplaced yes)
-		(property "Reference" "R20"
+		(property "Reference" "R19"
 			(at 44.45 89.5349 0)
 			(effects
@@
 			(project ""
 				(path "/b4b2c88d-f6cd-4e60-862d-e21f68728580/5e5b27f8-7a4c-45d0-95f8-aff71797fcd3/21d0e59e-a5df-4633-9634-c7d789255f22"
-					(reference "R16")
+					(reference "R19")
 					(unit 1)
 				)
 				(path "/b4b2c88d-f6cd-4e60-862d-e21f68728580/5e5b27f8-7a4c-45d0-95f8-aff71797fcd3/3e22df28-91f0-4c0f-b958-7bfd7fe99c70"
-					(reference "R20")
+					(reference "R23")
 					(unit 1)
 				)
 				(path "/b4b2c88d-f6cd-4e60-862d-e21f68728580/5e5b27f8-7a4c-45d0-95f8-aff71797fcd3/87e2c931-24b0-464d-a54c-5e253d37e662"
-					(reference "R24")
+					(reference "R27")
 					(unit 1)
 				)
@@
 		(dnp no)
 		(fields_autoplaced yes)
-		(property "Reference" "R14"
+		(property "Reference" "R17"
 			(at 45.72 64.1349 0)
 			(effects
@@
 			(project "sci_board"
 				(path "/b4b2c88d-f6cd-4e60-862d-e21f68728580/5e5b27f8-7a4c-45d0-95f8-aff71797fcd3/21d0e59e-a5df-4633-9634-c7d789255f22"
-					(reference "R14")
+					(reference "R17")
 					(unit 1)
 				)
 				(path "/b4b2c88d-f6cd-4e60-862d-e21f68728580/5e5b27f8-7a4c-45d0-95f8-aff71797fcd3/3e22df28-91f0-4c0f-b958-7bfd7fe99c70"
-					(reference "R18")
+					(reference "R21")
 					(unit 1)
 				)
 				(path "/b4b2c88d-f6cd-4e60-862d-e21f68728580/5e5b27f8-7a4c-45d0-95f8-aff71797fcd3/87e2c931-24b0-464d-a54c-5e253d37e662"
-					(reference "R22")
+					(reference "R25")
 					(unit 1)
 				)
@@
 		(dnp no)
 		(fields_autoplaced yes)
-		(property "Reference" "R15"
+		(property "Reference" "R18"
 			(at 62.23 64.1349 0)
 			(effects
@@
 			(project "sci_board"
 				(path "/b4b2c88d-f6cd-4e60-862d-e21f68728580/5e5b27f8-7a4c-45d0-95f8-aff71797fcd3/21d0e59e-a5df-4633-9634-c7d789255f22"
-					(reference "R15")
+					(reference "R18")
 					(unit 1)
 				)
 				(path "/b4b2c88d-f6cd-4e60-862d-e21f68728580/5e5b27f8-7a4c-45d0-95f8-aff71797fcd3/3e22df28-91f0-4c0f-b958-7bfd7fe99c70"
-					(reference "R19")
+					(reference "R22")
 					(unit 1)
 				)
 				(path "/b4b2c88d-f6cd-4e60-862d-e21f68728580/5e5b27f8-7a4c-45d0-95f8-aff71797fcd3/87e2c931-24b0-464d-a54c-5e253d37e662"
-					(reference "R23")
-					(unit 1)
-				)
+					(reference "R26")
+					(unit 1)
+				)

Commit message: tweaks before merge
Parts:
- J3: footprint Project:100519222410EHLF -> Common:100519222410EHLF
- NT1: footprint Project:NetTie-2_SMD_Pad0.3mm -> Common:NetTie-2_SMD_Pad0.3mm

Commit message: local switches and monitors for SCI and RF
Parts:
- renumbered R17 to R20, R18 to R21, R19 to R22, R20 to R23
Changed lines of the file:
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@@
 		(dnp no)
 		(fields_autoplaced yes)
-		(property "Reference" "R20"
+		(property "Reference" "R23"
 			(at 59.055 89.5349 0)
 			(effects
@@
 			(project "sci_board"
 				(path "/b4b2c88d-f6cd-4e60-862d-e21f68728580/5e5b27f8-7a4c-45d0-95f8-aff71797fcd3/21d0e59e-a5df-4633-9634-c7d789255f22"
-					(reference "R20")
+					(reference "R23")
 					(unit 1)
 				)
 				(path "/b4b2c88d-f6cd-4e60-862d-e21f68728580/5e5b27f8-7a4c-45d0-95f8-aff71797fcd3/3e22df28-91f0-4c0f-b958-7bfd7fe99c70"
-					(reference "R24")
+					(reference "R27")
 					(unit 1)
 				)
 				(path "/b4b2c88d-f6cd-4e60-862d-e21f68728580/5e5b27f8-7a4c-45d0-95f8-aff71797fcd3/87e2c931-24b0-464d-a54c-5e253d37e662"
-					(reference "R28")
+					(reference "R31")
 					(unit 1)
 				)
@@
 		(dnp no)
 		(fields_autoplaced yes)
-		(property "Reference" "R19"
+		(property "Reference" "R22"
 			(at 44.45 89.5349 0)
 			(effects
@@
 			(project ""
 				(path "/b4b2c88d-f6cd-4e60-862d-e21f68728580/5e5b27f8-7a4c-45d0-95f8-aff71797fcd3/21d0e59e-a5df-4633-9634-c7d789255f22"
-					(reference "R19")
+					(reference "R22")
 					(unit 1)
 				)
 				(path "/b4b2c88d-f6cd-4e60-862d-e21f68728580/5e5b27f8-7a4c-45d0-95f8-aff71797fcd3/3e22df28-91f0-4c0f-b958-7bfd7fe99c70"
-					(reference "R23")
+					(reference "R26")
 					(unit 1)
 				)
 				(path "/b4b2c88d-f6cd-4e60-862d-e21f68728580/5e5b27f8-7a4c-45d0-95f8-aff71797fcd3/87e2c931-24b0-464d-a54c-5e253d37e662"
-					(reference "R27")
+					(reference "R30")
 					(unit 1)
 				)
@@
 		(dnp no)
 		(fields_autoplaced yes)
-		(property "Reference" "R17"
+		(property "Reference" "R20"
 			(at 45.72 64.1349 0)
 			(effects
@@
 			(project "sci_board"
 				(path "/b4b2c88d-f6cd-4e60-862d-e21f68728580/5e5b27f8-7a4c-45d0-95f8-aff71797fcd3/21d0e59e-a5df-4633-9634-c7d789255f22"
-					(reference "R17")
+					(reference "R20")
 					(unit 1)
 				)
 				(path "/b4b2c88d-f6cd-4e60-862d-e21f68728580/5e5b27f8-7a4c-45d0-95f8-aff71797fcd3/3e22df28-91f0-4c0f-b958-7bfd7fe99c70"
-					(reference "R21")
+					(reference "R24")
 					(unit 1)
 				)
 				(path "/b4b2c88d-f6cd-4e60-862d-e21f68728580/5e5b27f8-7a4c-45d0-95f8-aff71797fcd3/87e2c931-24b0-464d-a54c-5e253d37e662"
-					(reference "R25")
+					(reference "R28")
 					(unit 1)
 				)
@@
 		(dnp no)
 		(fields_autoplaced yes)
-		(property "Reference" "R18"
+		(property "Reference" "R21"
 			(at 62.23 64.1349 0)
 			(effects
@@
 			(project "sci_board"
 				(path "/b4b2c88d-f6cd-4e60-862d-e21f68728580/5e5b27f8-7a4c-45d0-95f8-aff71797fcd3/21d0e59e-a5df-4633-9634-c7d789255f22"
-					(reference "R18")
+					(reference "R21")
 					(unit 1)
 				)
 				(path "/b4b2c88d-f6cd-4e60-862d-e21f68728580/5e5b27f8-7a4c-45d0-95f8-aff71797fcd3/3e22df28-91f0-4c0f-b958-7bfd7fe99c70"
-					(reference "R22")
+					(reference "R25")
 					(unit 1)
 				)
 				(path "/b4b2c88d-f6cd-4e60-862d-e21f68728580/5e5b27f8-7a4c-45d0-95f8-aff71797fcd3/87e2c931-24b0-464d-a54c-5e253d37e662"
-					(reference "R26")
-					(unit 1)
-				)
+					(reference "R29")
+					(unit 1)
+				)
