File: sci_board/cameras.kicad_sch (KiCad schematic)
At the start: 10 parts, among them J8 10051922-2410EHLF, X1 24MHz

Commit message: clenup BOM for SCI and AUX
Parts:
- J8: Manufacturer (none) -> Amphenol; Part Number (none) -> 10051922-2410EHLF
- R33: Part Number RT0402BRD07182KL -> RC0402FR-07182KL; Tolerance 0.1 -> 1
Changed lines of the file:
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@@
+			)
+		)
+		(property "Part Number" "10051922-2410EHLF"
+			(at 270.51 156.21 0)
+			(effects
+				(font
+					(size 1.27 1.27)
+				)
+				(hide yes)
+			)
+		)
+		(property "Manufacturer" "Amphenol"
+			(at 270.51 156.21 0)
+			(effects
+				(font
+					(size 1.27 1.27)
+				)
+				(hide yes)
 			)
 		)
@@
 			)
 		)
-		(property "Datasheet" "https://www.yageo.com/upload/media/product/app/datasheet/rchip/pyu-rt_1-to-0.01_rohs_l.pdf"
+		(property "Datasheet" "https://www.yageo.com/upload/media/product/products/datasheet/rchip/PYu-RC_Group_51_RoHS_L_12.pdf"
 			(at 247.015 78.74 0)
 			(effects
@@
 			)
 		)
-		(property "Part Number" "RT0402BRD07182KL"
+		(property "Part Number" "RC0402FR-07182KL"
 			(at 247.015 78.74 0)
 			(effects
@@
 			)
 		)
-		(property "Tolerance" "0.1"
+		(property "Tolerance" "1"
 			(at 247.015 78.74 0)
 			(effects

Commit message: cleaning up bom: remove main camera port since it has not pullups and capacitors, correcting some errors in camera switch
Parts:
- removed J8: 10051922-2410EHLF, Project:100519222410EHLF, symbol Project:10051922-2410EHLF
- removed JP7, JP8: SolderJumper_3_Open, Jumper:SolderJumper-3_P2.0mm_Open_TrianglePad1.0x1.5mm, symbol Jumper:SolderJumper_3_Open
- removed NT4: NetTie_2, Project:NetTie-2_SMD_Pad0.3mm, symbol Device:NetTie_2
- renumbered R32 to R38, R33 to R39

Commit message: local switches and monitors for SCI and RF
Parts:
- renumbered R38 to R41, R39 to R42
Changed lines of the file:
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@@
 		(on_board yes)
 		(dnp no)
-		(property "Reference" "R38"
+		(property "Reference" "R41"
 			(at 201.93 81.28 90)
 			(effects
@@
 			(project "sci_board"
 				(path "/b4b2c88d-f6cd-4e60-862d-e21f68728580/5e5b27f8-7a4c-45d0-95f8-aff71797fcd3"
-					(reference "R38")
+					(reference "R41")
 					(unit 1)
 				)
@@
 		(on_board yes)
 		(dnp no)
-		(property "Reference" "R39"
+		(property "Reference" "R42"
 			(at 246.38 81.28 90)
 			(effects
@@
 			(project "sci_board"
 				(path "/b4b2c88d-f6cd-4e60-862d-e21f68728580/5e5b27f8-7a4c-45d0-95f8-aff71797fcd3"
-					(reference "R39")
+					(reference "R42")
 					(unit 1)
 				)
