File: sci_board/dual_switch.kicad_sch (KiCad schematic)
At the start: 7 parts, among them U10 MIC2009YM6-TR, U11 MIC2009YM6-TR, U12 MIC2009YM6-TR

Commit message: tweaking SCI and AUX for production, using common sheets as much as possible
Parts:
- renumbered R26 to R28, R27 to R29, R28 to R30, R29 to R31
Changed lines of the file:
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@@
 		(dnp no)
 		(fields_autoplaced yes)
-		(property "Reference" "R27"
+		(property "Reference" "R29"
 			(at 201.295 81.2799 0)
 			(effects
@@
 			(project "sci_board"
 				(path "/b4b2c88d-f6cd-4e60-862d-e21f68728580/5e5b27f8-7a4c-45d0-95f8-aff71797fcd3/09c52fbd-a66a-456f-a3b3-a583ddfe7084"
-					(reference "R27")
+					(reference "R29")
 					(unit 1)
 				)
 				(path "/b4b2c88d-f6cd-4e60-862d-e21f68728580/5e5b27f8-7a4c-45d0-95f8-aff71797fcd3/3113fc14-4b9f-4852-8ddb-4c564d791d7f"
-					(reference "R19")
+					(reference "R21")
 					(unit 1)
 				)
 				(path "/b4b2c88d-f6cd-4e60-862d-e21f68728580/5e5b27f8-7a4c-45d0-95f8-aff71797fcd3/df99859d-8e37-4f21-a1c5-637d9e74b907"
-					(reference "R23")
+					(reference "R25")
 					(unit 1)
 				)
@@
 		(dnp no)
 		(fields_autoplaced yes)
-		(property "Reference" "R26"
+		(property "Reference" "R28"
 			(at 114.3 67.3099 0)
 			(effects
@@
 			(project "sci_board"
 				(path "/b4b2c88d-f6cd-4e60-862d-e21f68728580/5e5b27f8-7a4c-45d0-95f8-aff71797fcd3/09c52fbd-a66a-456f-a3b3-a583ddfe7084"
-					(reference "R26")
+					(reference "R28")
 					(unit 1)
 				)
 				(path "/b4b2c88d-f6cd-4e60-862d-e21f68728580/5e5b27f8-7a4c-45d0-95f8-aff71797fcd3/3113fc14-4b9f-4852-8ddb-4c564d791d7f"
-					(reference "R18")
+					(reference "R20")
 					(unit 1)
 				)
 				(path "/b4b2c88d-f6cd-4e60-862d-e21f68728580/5e5b27f8-7a4c-45d0-95f8-aff71797fcd3/df99859d-8e37-4f21-a1c5-637d9e74b907"
-					(reference "R22")
+					(reference "R24")
 					(unit 1)
 				)
@@
 		(dnp no)
 		(fields_autoplaced yes)
-		(property "Reference" "R28"
+		(property "Reference" "R30"
 			(at 133.35 81.9149 0)
 			(effects
@@
 			(project "sci_board"
 				(path "/b4b2c88d-f6cd-4e60-862d-e21f68728580/5e5b27f8-7a4c-45d0-95f8-aff71797fcd3/09c52fbd-a66a-456f-a3b3-a583ddfe7084"
-					(reference "R28")
+					(reference "R30")
 					(unit 1)
 				)
 				(path "/b4b2c88d-f6cd-4e60-862d-e21f68728580/5e5b27f8-7a4c-45d0-95f8-aff71797fcd3/3113fc14-4b9f-4852-8ddb-4c564d791d7f"
-					(reference "R20")
+					(reference "R22")
 					(unit 1)
 				)
 				(path "/b4b2c88d-f6cd-4e60-862d-e21f68728580/5e5b27f8-7a4c-45d0-95f8-aff71797fcd3/df99859d-8e37-4f21-a1c5-637d9e74b907"
-					(reference "R24")
+					(reference "R26")
 					(unit 1)
 				)
@@
 		(dnp no)
 		(fields_autoplaced yes)
-		(property "Reference" "R29"
+		(property "Reference" "R31"
 			(at 61.595 82.5499 0)
 			(effects
@@
 			(project "sci_board"
 				(path "/b4b2c88d-f6cd-4e60-862d-e21f68728580/5e5b27f8-7a4c-45d0-95f8-aff71797fcd3/09c52fbd-a66a-456f-a3b3-a583ddfe7084"
-					(reference "R29")
+					(reference "R31")
 					(unit 1)
 				)
 				(path "/b4b2c88d-f6cd-4e60-862d-e21f68728580/5e5b27f8-7a4c-45d0-95f8-aff71797fcd3/3113fc14-4b9f-4852-8ddb-4c564d791d7f"
-					(reference "R21")
+					(reference "R23")
 					(unit 1)
 				)
 				(path "/b4b2c88d-f6cd-4e60-862d-e21f68728580/5e5b27f8-7a4c-45d0-95f8-aff71797fcd3/df99859d-8e37-4f21-a1c5-637d9e74b907"
-					(reference "R25")
-					(unit 1)
-				)
+					(reference "R27")
+					(unit 1)
+				)

Commit message: clenup BOM for SCI and AUX
Parts:
- R28: value 10K -> 100K; Part Number RC0402FR-0710KL -> RC0402FR-07100KL
Changed lines of the file:
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@@
 			)
 		)
-		(property "Value" "10K"
+		(property "Value" "100K"
 			(at 114.3 69.8499 0)
 			(effects
@@
 			)
 		)
-		(property "Part Number" "RC0402FR-0710KL"
+		(property "Part Number" "RC0402FR-07100KL"
 			(at 111.76 68.58 0)
 			(effects

Commit message: cleaning up bom: remove main camera port since it has not pullups and capacitors, correcting some errors in camera switch
Parts:
- R35: renamed from R29; value 1K5 -> 988R; Part Number RC0603FR-071K5L -> RT0603DRE07988RL
- R36: renamed from R30; value 1K5 -> 988R; Part Number RC0603FR-071K5L -> RT0603DRE07988RL
- R37: renamed from R31; value 1K5 -> 988R; Part Number RC0603FR-071K5L -> RT0603DRE07988RL
- U10, U11, U12: value MIC2009YM6-TR -> MIC2009A-1YM6-TR; Part Number MIC2009YM6-TR -> SOT-23-6 MIC2009A-1YM6-TR
- renumbered R28 to R34
Other:
- note added: "OUT RSET LIM_MIN LIM_MAX 0.1A 1928Ω 0.063A 0.136A 0.2A 993Ω 0.137A 0.265A 0.3A 673Ω 0.216A 0.391A 0.4A 511Ω 0.296A 0.515A 0.5A 413Ω 0.379A 0.637A 0.6A 346Ω 0.463A 0.759A 0.7A 299Ω 0.548A 0.880A 0.8A 263Ω 0.634A 1.001A 0.9A 235Ω 0.722A 1.121A"
Changed lines of the file:
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@@
+		)
+	)
+	(text "OUT  RSET  LIM_MIN LIM_MAX\n0.1A 1928Ω 0.063A  0.136A\n0.2A 993Ω  0.137A  0.265A\n0.3A 673Ω  0.216A  0.391A\n0.4A 511Ω  0.296A  0.515A\n0.5A 413Ω  0.379A  0.637A\n0.6A 346Ω  0.463A  0.759A\n0.7A 299Ω  0.548A  0.880A\n0.8A 263Ω  0.634A  1.001A\n0.9A 235Ω  0.722A  1.121A"
+		(exclude_from_sim no)
+		(at 63.5 101.6 0)
+		(effects
+			(font
+				(size 1.27 1.27)
+			)
+			(justify left)
 		)
 	)
@@
 			)
 		)
-		(property "Value" "MIC2009YM6-TR"
+		(property "Value" "MIC2009A-1YM6-TR"
 			(at 78.105 64.135 0)
 			(effects
@@
 			)
 		)
-		(property "Part Number" "MIC2009YM6-TR"
+		(property "Part Number" "SOT-23-6 MIC2009A-1YM6-TR"
 			(at 59.055 69.85 0)
 			(effects
@@
 		(dnp no)
 		(fields_autoplaced yes)
-		(property "Reference" "R29"
-			(at 201.295 81.2799 0)
+		(property "Reference" "R35"
+			(at 200.66 81.2799 0)
 			(effects
 				(font
@@
 			)
 		)
-		(property "Value" "1K5"
-			(at 201.295 83.8199 0)
+		(property "Value" "988R"
+			(at 200.66 83.8199 0)
 			(effects
 				(font
@@
 			)
 		)
-		(property "Datasheet" "https://www.yageo.com/upload/media/product/products/datasheet/rchip/PYu-RC_Group_51_RoHS_L_12.pdf"
+		(property "Datasheet" "https://www.yageo.com/upload/media/product/app/datasheet/rchip/pyu-rt_1-to-0.01_rohs_l.pdf"
 			(at 198.755 82.55 0)
 			(effects
@@
 			)
 		)
-		(property "Part Number" "RC0603FR-071K5L"
+		(property "Part Number" "RT0603DRE07988RL"
 			(at 198.755 82.55 0)
 			(effects
@@
 			(project "sci_board"
 				(path "/b4b2c88d-f6cd-4e60-862d-e21f68728580/5e5b27f8-7a4c-45d0-95f8-aff71797fcd3/09c52fbd-a66a-456f-a3b3-a583ddfe7084"
-					(reference "R29")
+					(reference "R35")
 					(unit 1)
 				)
 				(path "/b4b2c88d-f6cd-4e60-862d-e21f68728580/5e5b27f8-7a4c-45d0-95f8-aff71797fcd3/3113fc14-4b9f-4852-8ddb-4c564d791d7f"
-					(reference "R21")
+					(reference "R27")
 					(unit 1)
 				)
 				(path "/b4b2c88d-f6cd-4e60-862d-e21f68728580/5e5b27f8-7a4c-45d0-95f8-aff71797fcd3/df99859d-8e37-4f21-a1c5-637d9e74b907"
-					(reference "R25")
+					(reference "R31")
 					(unit 1)
 				)
@@
 			)
 		)
-		(property "Value" "MIC2009YM6-TR"
+		(property "Value" "MIC2009A-1YM6-TR"
 			(at 149.86 63.5 0)
 			(effects
@@
 			)
 		)
-		(property "Part Number" "MIC2009YM6-TR"
+		(property "Part Number" "SOT-23-6 MIC2009A-1YM6-TR"
 			(at 130.81 69.215 0)
 			(effects
@@
 		(dnp no)
 		(fields_autoplaced yes)
-		(property "Reference" "R28"
+		(property "Reference" "R34"
 			(at 114.3 67.3099 0)
 			(effects
@@
 			(project "sci_board"
 				(path "/b4b2c88d-f6cd-4e60-862d-e21f68728580/5e5b27f8-7a4c-45d0-95f8-aff71797fcd3/09c52fbd-a66a-456f-a3b3-a583ddfe7084"
-					(reference "R28")
+					(reference "R34")
 					(unit 1)
 				)
 				(path "/b4b2c88d-f6cd-4e60-862d-e21f68728580/5e5b27f8-7a4c-45d0-95f8-aff71797fcd3/3113fc14-4b9f-4852-8ddb-4c564d791d7f"
-					(reference "R20")
+					(reference "R26")
 					(unit 1)
 				)
 				(path "/b4b2c88d-f6cd-4e60-862d-e21f68728580/5e5b27f8-7a4c-45d0-95f8-aff71797fcd3/df99859d-8e37-4f21-a1c5-637d9e74b907"
-					(reference "R24")
+					(reference "R30")
 					(unit 1)
 				)
@@
 			)
 		)
-		(property "Value" "MIC2009YM6-TR"
+		(property "Value" "MIC2009A-1YM6-TR"
 			(at 217.805 62.865 0)
 			(effects
@@
 			)
 		)
-		(property "Part Number" "MIC2009YM6-TR"
+		(property "Part Number" "SOT-23-6 MIC2009A-1YM6-TR"
 			(at 198.755 68.58 0)
 			(effects
@@
 		(dnp no)
 		(fields_autoplaced yes)
-		(property "Reference" "R30"
+		(property "Reference" "R36"
 			(at 133.35 81.9149 0)
 			(effects
@@
 			)
 		)
-		(property "Value" "1K5"
+		(property "Value" "988R"
 			(at 133.35 84.4549 0)
 			(effects
@@
 			)
 		)
-		(property "Datasheet" "https://www.yageo.com/upload/media/product/products/datasheet/rchip/PYu-RC_Group_51_RoHS_L_12.pdf"
+		(property "Datasheet" "https://www.yageo.com/upload/media/product/app/datasheet/rchip/pyu-rt_1-to-0.01_rohs_l.pdf"
 			(at 130.81 83.185 0)
 			(effects
@@
 			)
 		)
-		(property "Part Number" "RC0603FR-071K5L"
+		(property "Part Number" "RT0603DRE07988RL"
 			(at 130.81 83.185 0)
 			(effects
@@
 			(project "sci_board"
 				(path "/b4b2c88d-f6cd-4e60-862d-e21f68728580/5e5b27f8-7a4c-45d0-95f8-aff71797fcd3/09c52fbd-a66a-456f-a3b3-a583ddfe7084"
-					(reference "R30")
+					(reference "R36")
 					(unit 1)
 				)
 				(path "/b4b2c88d-f6cd-4e60-862d-e21f68728580/5e5b27f8-7a4c-45d0-95f8-aff71797fcd3/3113fc14-4b9f-4852-8ddb-4c564d791d7f"
-					(reference "R22")
+					(reference "R28")
 					(unit 1)
 				)
 				(path "/b4b2c88d-f6cd-4e60-862d-e21f68728580/5e5b27f8-7a4c-45d0-95f8-aff71797fcd3/df99859d-8e37-4f21-a1c5-637d9e74b907"
-					(reference "R26")
+					(reference "R32")
 					(unit 1)
 				)
@@
 		(dnp no)
 		(fields_autoplaced yes)
-		(property "Reference" "R31"
-			(at 61.595 82.5499 0)
+		(property "Reference" "R37"
+			(at 60.96 82.5499 0)
 			(effects
 				(font
@@
 			)
 		)
-		(property "Value" "1K5"
-			(at 61.595 85.0899 0)
+		(property "Value" "988R"
+			(at 60.96 85.0899 0)
 			(effects
 				(font
@@
 			)
 		)
-		(property "Datasheet" "https://www.yageo.com/upload/media/product/products/datasheet/rchip/PYu-RC_Group_51_RoHS_L_12.pdf"
+		(property "Datasheet" "https://www.yageo.com/upload/media/product/app/datasheet/rchip/pyu-rt_1-to-0.01_rohs_l.pdf"
 			(at 59.055 83.82 0)
 			(effects
@@
 			)
 		)
-		(property "Part Number" "RC0603FR-071K5L"
+		(property "Part Number" "RT0603DRE07988RL"
 			(at 59.055 83.82 0)
 			(effects
@@
 			(project "sci_board"
 				(path "/b4b2c88d-f6cd-4e60-862d-e21f68728580/5e5b27f8-7a4c-45d0-95f8-aff71797fcd3/09c52fbd-a66a-456f-a3b3-a583ddfe7084"
-					(reference "R31")
+					(reference "R37")
 					(unit 1)
 				)
 				(path "/b4b2c88d-f6cd-4e60-862d-e21f68728580/5e5b27f8-7a4c-45d0-95f8-aff71797fcd3/3113fc14-4b9f-4852-8ddb-4c564d791d7f"
-					(reference "R23")
+					(reference "R29")
 					(unit 1)
 				)
 				(path "/b4b2c88d-f6cd-4e60-862d-e21f68728580/5e5b27f8-7a4c-45d0-95f8-aff71797fcd3/df99859d-8e37-4f21-a1c5-637d9e74b907"
-					(reference "R27")
-					(unit 1)
-				)
+					(reference "R33")
+					(unit 1)
+				)

Commit message: QC, add second 3V regulator to AUX, INT pullups on AUX SCI AVI
Parts:
- removed R34: 100K, Resistor_SMD:R_0402_1005Metric_Pad0.72x0.64mm_HandSolder, symbol Device:R
Changed lines of the file:
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@@
 	(paper "A4")
-	(junction
-		(at 111.76 72.39)
-		(diameter 0)
-		(color 0 0 0 0)
-	)
 	(junction
 		(at 182.245 96.52)
@@
 			)
 			(justify left)
-		)
-	)
-	(hierarchical_label "VIN3"
-		(shape input)
-		(at 111.76 64.77 180)
-		(fields_autoplaced yes)
-		(effects
-			(font
-				(size 1.27 1.27)
-			)
-			(justify right)
 		)
 	)
@@
 				)
 				(path "/b4b2c88d-f6cd-4e60-862d-e21f68728580/5e5b27f8-7a4c-45d0-95f8-aff71797fcd3/3113fc14-4b9f-4852-8ddb-4c564d791d7f"
-					(reference "R27")
+					(reference "R29")
 					(unit 1)
 				)
 				(path "/b4b2c88d-f6cd-4e60-862d-e21f68728580/5e5b27f8-7a4c-45d0-95f8-aff71797fcd3/df99859d-8e37-4f21-a1c5-637d9e74b907"
-					(reference "R31")
+					(reference "R32")
 					(unit 1)
 				)
@@
 	)
 	(symbol
-		(lib_id "Device:R")
-		(at 111.76 68.58 0)
-		(unit 1)
-		(exclude_from_sim no)
-		(in_bom yes)
-		(on_board yes)
-		(dnp no)
-		(fields_autoplaced yes)
-		(property "Reference" "R34"
-			(at 114.3 67.3099 0)
-			(effects
-				(font
-					(size 1.27 1.27)
-				)
-				(justify left)
-			)
-		)
-		(property "Value" "100K"
-			(at 114.3 69.8499 0)
-			(effects
-				(font
-					(size 1.27 1.27)
-				)
-				(justify left)
-			)
-		)
-		(property "Footprint" "Resistor_SMD:R_0402_1005Metric_Pad0.72x0.64mm_HandSolder"
-			(at 109.982 68.58 90)
-			(effects
-				(font
-					(size 1.27 1.27)
-				)
-				(hide yes)
-			)
-		)
-		(property "Datasheet" "https://www.yageo.com/upload/media/product/products/datasheet/rchip/PYu-RC_Group_51_RoHS_L_12.pdf"
-			(at 111.76 68.58 0)
-			(effects
-				(font
-					(size 1.27 1.27)
-				)
-				(hide yes)
-			)
-		)
-		(property "Description" "Resistor"
-			(at 111.76 68.58 0)
-			(effects
-				(font
-					(size 1.27 1.27)
-				)
-				(hide yes)
-			)
-		)
-		(property "Manufacturer" "YAGEO"
-			(at 111.76 68.58 0)
-			(effects
-				(font
-					(size 1.27 1.27)
-				)
-				(hide yes)
-			)
-		)
-		(property "Note" "INT pullup"
-			(at 111.76 68.58 0)
-			(effects
-				(font
-					(size 1.27 1.27)
-				)
-				(hide yes)
-			)
-		)
-		(property "Part Number" "RC0402FR-07100KL"
-			(at 111.76 68.58 0)
-			(effects
-				(font
-					(size 1.27 1.27)
-				)
-				(hide yes)
-			)
-		)
-		(property "Tolerance" "1"
-			(at 111.76 68.58 0)
-			(effects
-				(font
-					(size 1.27 1.27)
-				)
-				(hide yes)
-			)
-		)
-		(pin "1"
-		)
-		(pin "2"
-		)
-		(instances
-			(project "sci_board"
-				(path "/b4b2c88d-f6cd-4e60-862d-e21f68728580/5e5b27f8-7a4c-45d0-95f8-aff71797fcd3/09c52fbd-a66a-456f-a3b3-a583ddfe7084"
-					(reference "R34")
-					(unit 1)
-				)
-				(path "/b4b2c88d-f6cd-4e60-862d-e21f68728580/5e5b27f8-7a4c-45d0-95f8-aff71797fcd3/3113fc14-4b9f-4852-8ddb-4c564d791d7f"
-					(reference "R26")
-					(unit 1)
-				)
-				(path "/b4b2c88d-f6cd-4e60-862d-e21f68728580/5e5b27f8-7a4c-45d0-95f8-aff71797fcd3/df99859d-8e37-4f21-a1c5-637d9e74b907"
-					(reference "R30")
-					(unit 1)
-				)
-			)
-		)
-	)
-	(symbol
 		(lib_id "Project:MIC2009YM6-TR")
 		(at 198.755 68.58 0)
@@
 				)
 				(path "/b4b2c88d-f6cd-4e60-862d-e21f68728580/5e5b27f8-7a4c-45d0-95f8-aff71797fcd3/3113fc14-4b9f-4852-8ddb-4c564d791d7f"
-					(reference "R28")
+					(reference "R30")
 					(unit 1)
 				)
 				(path "/b4b2c88d-f6cd-4e60-862d-e21f68728580/5e5b27f8-7a4c-45d0-95f8-aff71797fcd3/df99859d-8e37-4f21-a1c5-637d9e74b907"
-					(reference "R32")
+					(reference "R33")
 					(unit 1)
 				)
@@
 				)
 				(path "/b4b2c88d-f6cd-4e60-862d-e21f68728580/5e5b27f8-7a4c-45d0-95f8-aff71797fcd3/3113fc14-4b9f-4852-8ddb-4c564d791d7f"
-					(reference "R29")
+					(reference "R31")
 					(unit 1)
 				)
 				(path "/b4b2c88d-f6cd-4e60-862d-e21f68728580/5e5b27f8-7a4c-45d0-95f8-aff71797fcd3/df99859d-8e37-4f21-a1c5-637d9e74b907"
-					(reference "R33")
-					(unit 1)
-				)
+					(reference "R34")
+					(unit 1)
+				)

Commit message: local switches and monitors for SCI and RF
Parts:
- renumbered R35 to R38, R36 to R39, R37 to R40
Changed lines of the file:
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@@
 		(dnp no)
 		(fields_autoplaced yes)
-		(property "Reference" "R35"
+		(property "Reference" "R38"
 			(at 200.66 81.2799 0)
 			(effects
@@
 			(project "sci_board"
 				(path "/b4b2c88d-f6cd-4e60-862d-e21f68728580/5e5b27f8-7a4c-45d0-95f8-aff71797fcd3/09c52fbd-a66a-456f-a3b3-a583ddfe7084"
+					(reference "R38")
+					(unit 1)
+				)
+				(path "/b4b2c88d-f6cd-4e60-862d-e21f68728580/5e5b27f8-7a4c-45d0-95f8-aff71797fcd3/3113fc14-4b9f-4852-8ddb-4c564d791d7f"
+					(reference "R32")
+					(unit 1)
+				)
+				(path "/b4b2c88d-f6cd-4e60-862d-e21f68728580/5e5b27f8-7a4c-45d0-95f8-aff71797fcd3/df99859d-8e37-4f21-a1c5-637d9e74b907"
 					(reference "R35")
-					(unit 1)
-				)
-				(path "/b4b2c88d-f6cd-4e60-862d-e21f68728580/5e5b27f8-7a4c-45d0-95f8-aff71797fcd3/3113fc14-4b9f-4852-8ddb-4c564d791d7f"
-					(reference "R29")
-					(unit 1)
-				)
-				(path "/b4b2c88d-f6cd-4e60-862d-e21f68728580/5e5b27f8-7a4c-45d0-95f8-aff71797fcd3/df99859d-8e37-4f21-a1c5-637d9e74b907"
-					(reference "R32")
 					(unit 1)
 				)
@@
 		(dnp no)
 		(fields_autoplaced yes)
-		(property "Reference" "R36"
+		(property "Reference" "R39"
 			(at 133.35 81.9149 0)
 			(effects
@@
 			(project "sci_board"
 				(path "/b4b2c88d-f6cd-4e60-862d-e21f68728580/5e5b27f8-7a4c-45d0-95f8-aff71797fcd3/09c52fbd-a66a-456f-a3b3-a583ddfe7084"
+					(reference "R39")
+					(unit 1)
+				)
+				(path "/b4b2c88d-f6cd-4e60-862d-e21f68728580/5e5b27f8-7a4c-45d0-95f8-aff71797fcd3/3113fc14-4b9f-4852-8ddb-4c564d791d7f"
+					(reference "R33")
+					(unit 1)
+				)
+				(path "/b4b2c88d-f6cd-4e60-862d-e21f68728580/5e5b27f8-7a4c-45d0-95f8-aff71797fcd3/df99859d-8e37-4f21-a1c5-637d9e74b907"
 					(reference "R36")
-					(unit 1)
-				)
-				(path "/b4b2c88d-f6cd-4e60-862d-e21f68728580/5e5b27f8-7a4c-45d0-95f8-aff71797fcd3/3113fc14-4b9f-4852-8ddb-4c564d791d7f"
-					(reference "R30")
-					(unit 1)
-				)
-				(path "/b4b2c88d-f6cd-4e60-862d-e21f68728580/5e5b27f8-7a4c-45d0-95f8-aff71797fcd3/df99859d-8e37-4f21-a1c5-637d9e74b907"
-					(reference "R33")
 					(unit 1)
 				)
@@
 		(dnp no)
 		(fields_autoplaced yes)
-		(property "Reference" "R37"
+		(property "Reference" "R40"
 			(at 60.96 82.5499 0)
 			(effects
@@
 			(project "sci_board"
 				(path "/b4b2c88d-f6cd-4e60-862d-e21f68728580/5e5b27f8-7a4c-45d0-95f8-aff71797fcd3/09c52fbd-a66a-456f-a3b3-a583ddfe7084"
+					(reference "R40")
+					(unit 1)
+				)
+				(path "/b4b2c88d-f6cd-4e60-862d-e21f68728580/5e5b27f8-7a4c-45d0-95f8-aff71797fcd3/3113fc14-4b9f-4852-8ddb-4c564d791d7f"
+					(reference "R34")
+					(unit 1)
+				)
+				(path "/b4b2c88d-f6cd-4e60-862d-e21f68728580/5e5b27f8-7a4c-45d0-95f8-aff71797fcd3/df99859d-8e37-4f21-a1c5-637d9e74b907"
 					(reference "R37")
 					(unit 1)
 				)
-				(path "/b4b2c88d-f6cd-4e60-862d-e21f68728580/5e5b27f8-7a4c-45d0-95f8-aff71797fcd3/3113fc14-4b9f-4852-8ddb-4c564d791d7f"
-					(reference "R31")
-					(unit 1)
-				)
-				(path "/b4b2c88d-f6cd-4e60-862d-e21f68728580/5e5b27f8-7a4c-45d0-95f8-aff71797fcd3/df99859d-8e37-4f21-a1c5-637d9e74b907"
-					(reference "R34")
-					(unit 1)
-				)
