File: openlst-hw/openlst-hw.kicad_pcb (KiCad board)
At the start: 4 copper layers, 80 x 80 mm, 140 parts, among them J1 Conn_02x03_Pin, J10 Conn_01x06, J11 Conn_01x04, J13 10155435-00011LF, J14 Conn_01x03_Pin, J2 Conn_01x06_Pin, J3 Conn_01x03_Pin, J4 Conn_01x03_Pin, J5 SMA Jack, J6 Conn_01x03_Pin, J7 SMA Jack, J8 PC104 Conn_02x20_Odd_Even, J9 Conn_01x05_Pin, SW1 EVP-AA602W, SW2 EVP-AA602W, U1 CC1110, U10 STM32L496RGTx, U11 74LVC2G07, U2 MIC803, U3 SF2446E, U4 PE4250MLI, U5 PE4250MLI, U6 0433BM15A0001, U7 RFFM6406, U8 TCAN3414, U9 TCAN3414, X1 27MHz, X2 10MHz

Commit message: propate the changes to RF
Parts:
- removed the C58 at (75.1, 112.3)
- removed the J13 at (100.1, 137.1)
- removed the R25 at (120.0, 124.4)
- removed the R26 at (120.0, 122.7)
- removed the R27 at (120.0, 121.1)
- added C59: 100nF, Capacitor_SMD:C_0402_1005Metric_Pad0.74x0.62mm_HandSolder, F.Cu at (74.9, 112.3)
- added J11: 10155435-00011LF, Common:AMPHENOL_10155435-00011LF, F.Cu at (100.1, 137.1)
- added R31: 1K, Resistor_SMD:R_0402_1005Metric_Pad0.72x0.64mm_HandSolder, F.Cu at (120.8, 124.4)
- added R32: 1K, Resistor_SMD:R_0402_1005Metric_Pad0.72x0.64mm_HandSolder, F.Cu at (120.8, 122.8)
- added R33: 1K, Resistor_SMD:R_0402_1005Metric_Pad0.72x0.64mm_HandSolder, F.Cu at (120.8, 121.1)
- added R36: 100K, Resistor_SMD:R_0402_1005Metric_Pad0.72x0.64mm_HandSolder, F.Cu at (74.0, 112.3)
- R26: renamed from R32; value 100K -> 300K
- R28: value 1K -> 100K
- R29: value 1K -> 5K1
- R30: value 10K -> 5K1
- R34, R35: value 5K1 -> 1K
- moved SW2 37.8 mm to (78.1, 112.3)
- moved SW1 37.8 mm to (115.6, 117.2), turned to 0 degrees
- moved R34 26.0 mm to (120.8, 119.4), turned to 0 degrees
- moved R29 25.9 mm to (97.6, 131.0), turned to 0 degrees
- moved R35 22.3 mm to (120.8, 117.8), turned to 0 degrees
- moved R30 16.6 mm to (102.7, 131.0), turned to 180 degrees
- moved R28 7.96 mm to (112.2, 117.5), turned to 90 degrees
- renumbered C59 to C58, J14 to J10, J10 to J12, J11 to J13, R31 to R25, R33 to R27
Connections:
- R28 pad 1: Net-(D8-A) -> /CAN Bridge/PMIC/BOOT
- R28 pad 2: /CAN Bridge/PMIC/LED4 -> GND
- R29 pad 1: Net-(D9-A) -> GND
- R29 pad 2: /CAN Bridge/PMIC/LED5 -> Net-(J11-CC1_A)
- R30 pad 1: /CAN Bridge/PMIC/BOOT -> GND
- R30 pad 2: GND -> Net-(J11-CC2_B)
- R34 pad 1: Net-(J13-CC1_A) -> /CAN Bridge/PMIC/LED4
- R34 pad 2: GND -> Net-(D8-A)
- R35 pad 1: GND -> /CAN Bridge/PMIC/LED5
- R35 pad 2: Net-(J13-CC2_B) -> Net-(D9-A)
- SW1 pad 1: unconnected-(SW1-Pad1) -> /INTERBOARD_CONNECTOR2/3V3_17_RF1_BRIDGE
- SW1 pad 2: unconnected-(SW1-Pad2) -> /CAN Bridge/PMIC/BOOT
- SW1 pad 3: /CAN Bridge/PMIC/Schmitt Trigger/IN2 -> unconnected-(SW1-Pad3)
- SW1 pad 4: GND -> unconnected-(SW1-Pad4)
- SW2 pad 3: /INTERBOARD_CONNECTOR2/3V3_17_RF1_BRIDGE -> /CAN Bridge/PMIC/RESET/RESET
- SW2 pad 4: /CAN Bridge/PMIC/BOOT -> GND
- U10 pad 44: /CAN Bridge/PMIC/USB/USB_OTG_FS_DM -> /CAN Bridge/PMIC/USB/DN
- U10 pad 45: /CAN Bridge/PMIC/USB/USB_OTG_FS_DP -> /CAN Bridge/PMIC/USB/DP
- U11 pad 3: /CAN Bridge/PMIC/Schmitt Trigger/IN2 -> /CAN Bridge/PMIC/RESET/RESET
Routing:
- net /INTERBOARD_CONNECTOR2/3V3_17_RF1_BRIDGE: track 92.3 -> 54.7 mm, vias 14 -> 15
- net /CAN Bridge/PMIC/USB/USB_OTG_FS_DM: track 11.5 -> 0.00 mm
- net /CAN Bridge/PMIC/USB/DN: track 0.00 -> 11.4 mm
- net /CAN Bridge/PMIC/USB/DP: track 0.00 -> 10.9 mm
- net /CAN Bridge/PMIC/USB/USB_OTG_FS_DP: track 10.6 -> 0.00 mm
- net /INTERBOARD_CONNECTOR2/3V3_18_RF1_COMM: track 63.3 -> 57.3 mm
- net /CAN Bridge/PMIC/RESET/RESET: track 0.00 -> 4.88 mm
- net /CAN Bridge/PMIC/Schmitt Trigger/IN2: track 3.91 -> 0.00 mm
- net Net-(J13-CC1_A): track 1.69 -> 0.00 mm
- net Net-(J13-CC2_B): track 1.62 -> 0.00 mm
- net Net-(J11-CC1_A): track 0.00 -> 1.59 mm
- net Net-(J11-CC2_B): track 0.00 -> 1.43 mm
- net Net-(D7-A): track 2.39 -> 1.40 mm
- net Net-(D6-A): track 2.36 -> 1.38 mm
- net Net-(D5-A): track 2.34 -> 1.41 mm
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
Commit message: local switches and monitors for SCI and RF
Parts:
- added C48: 100nF, Capacitor_SMD:C_0402_1005Metric_Pad0.74x0.62mm_HandSolder, F.Cu at (118.0, 106.0)
- added C49: 100nF, Capacitor_SMD:C_0402_1005Metric_Pad0.74x0.62mm_HandSolder, F.Cu at (119.9, 134.4)
- added C50: 10uF, Capacitor_SMD:C_0603_1608Metric_Pad1.08x0.95mm_HandSolder, F.Cu at (119.6, 128.5)
- added C51: 10uF, Capacitor_SMD:C_0603_1608Metric_Pad1.08x0.95mm_HandSolder, F.Cu at (121.5, 132.3)
- added C52: 100nF, Capacitor_SMD:C_0402_1005Metric_Pad0.74x0.62mm_HandSolder, F.Cu at (135.1, 115.1)
- added C53: 10uF, Capacitor_SMD:C_0603_1608Metric_Pad1.08x0.95mm_HandSolder, F.Cu at (129.2, 115.4)
- added C54: 10uF, Capacitor_SMD:C_0603_1608Metric_Pad1.08x0.95mm_HandSolder, F.Cu at (132.9, 113.5)
- added C65: 100nF, Capacitor_SMD:C_0402_1005Metric_Pad0.74x0.62mm_HandSolder, F.Cu at (123.3, 105.9)
- added C66: 10uF, Capacitor_SMD:C_0603_1608Metric_Pad1.08x0.95mm_HandSolder, F.Cu at (123.6, 111.8)
- added C67: 10uF, Capacitor_SMD:C_0603_1608Metric_Pad1.08x0.95mm_HandSolder, F.Cu at (121.7, 108.1)
- added C70: 100nF, Capacitor_SMD:C_0402_1005Metric_Pad0.74x0.62mm_HandSolder, F.Cu at (112.4, 125.5)
- added C71: 100nF, Capacitor_SMD:C_0402_1005Metric_Pad0.74x0.62mm_HandSolder, F.Cu at (107.3, 110.8)
- added C72: 100nF, Capacitor_SMD:C_0402_1005Metric_Pad0.74x0.62mm_HandSolder, F.Cu at (130.7, 131.4)
- added C73: 10uF, Capacitor_SMD:C_0603_1608Metric_Pad1.08x0.95mm_HandSolder, F.Cu at (130.3, 125.6)
- added C74: 10uF, Capacitor_SMD:C_0603_1608Metric_Pad1.08x0.95mm_HandSolder, F.Cu at (132.2, 129.3)
- added R23: 5K1, Resistor_SMD:R_0402_1005Metric_Pad0.72x0.64mm_HandSolder, F.Cu at (92.4, 121.2)
- added R24: 5K1, Resistor_SMD:R_0402_1005Metric_Pad0.72x0.64mm_HandSolder, F.Cu at (92.4, 122.1)
- added R27: 988R, Resistor_SMD:R_0603_1608Metric_Pad0.98x0.95mm_HandSolder, F.Cu at (129.7, 109.7)
- added R28: 988R, Resistor_SMD:R_0603_1608Metric_Pad0.98x0.95mm_HandSolder, F.Cu at (131.3, 121.5)
- added R29: 988R, Resistor_SMD:R_0603_1608Metric_Pad0.98x0.95mm_HandSolder, F.Cu at (124.3, 127.6)
- added R30: 988R, Resistor_SMD:R_0603_1608Metric_Pad0.98x0.95mm_HandSolder, F.Cu at (113.5, 130.6)
- added R31: 100K, Resistor_SMD:R_0402_1005Metric_Pad0.72x0.64mm_HandSolder, F.Cu at (114.7, 128.8)
- added R32: 10m, Resistor_SMD:R_0805_2012Metric_Pad1.20x1.40mm_HandSolder, F.Cu at (119.8, 132.1)
- added R33: 100K, Resistor_SMD:R_0402_1005Metric_Pad0.72x0.64mm_HandSolder, F.Cu at (129.4, 120.4)
- added R34: 10m, Resistor_SMD:R_0805_2012Metric_Pad1.20x1.40mm_HandSolder, F.Cu at (132.8, 115.2)
- added R36: 22R, Resistor_SMD:R_0402_1005Metric_Pad0.72x0.64mm_HandSolder, F.Cu at (108.5, 122.1)
- added R37: 22R, Resistor_SMD:R_0402_1005Metric_Pad0.72x0.64mm_HandSolder, F.Cu at (108.5, 120.8)
- added R39: 100K, Resistor_SMD:R_0402_1005Metric_Pad0.72x0.64mm_HandSolder, F.Cu at (128.5, 111.6)
- added R40: 10m, Resistor_SMD:R_0805_2012Metric_Pad1.20x1.40mm_HandSolder, F.Cu at (123.4, 108.3)
- added R51: 100K, Resistor_SMD:R_0402_1005Metric_Pad0.72x0.64mm_HandSolder, F.Cu at (115.8, 125.5)
- added R52: 100K, Resistor_SMD:R_0402_1005Metric_Pad0.72x0.64mm_HandSolder, F.Cu at (110.3, 123.4)
- added R53: 100K, Resistor_SMD:R_0402_1005Metric_Pad0.72x0.64mm_HandSolder, F.Cu at (118.7, 121.0)
- added R54: 22R, Resistor_SMD:R_0402_1005Metric_Pad0.72x0.64mm_HandSolder, F.Cu at (118.7, 123.2)
- added R55: 100K, Resistor_SMD:R_0402_1005Metric_Pad0.72x0.64mm_HandSolder, F.Cu at (125.5, 125.7)
- added R56: 10m, Resistor_SMD:R_0805_2012Metric_Pad1.20x1.40mm_HandSolder, F.Cu at (130.5, 129.1)
- added U10: MCP23008T-E/SS, Package_SO:SSOP-20_5.3x7.2mm_P0.65mm, F.Cu at (114.3, 110.3)
- added U11: MIC2009A-1YM6-TR, Common:SOT-23-6_Handsoldering, F.Cu at (117.0, 128.9)
- added U12: INA226AIDGSR, Common:SOP50P490X110-10N, F.Cu at (115.7, 133.1)
- added U13: MIC2009A-1YM6-TR, Common:SOT-23-6_Handsoldering, F.Cu at (129.7, 118.0)
- added U14: INA226AIDGSR, Common:SOP50P490X110-10N, F.Cu at (133.8, 119.3)
- added U16: MIC2009A-1YM6-TR, Common:SOT-23-6_Handsoldering, F.Cu at (126.2, 111.4)
- added U17: INA226AIDGSR, Common:SOP50P490X110-10N, F.Cu at (127.5, 107.2)
- added U19: MR25H10, Package_DFN_QFN:DFN-8-1EP_6x5mm_P1.27mm_EP2x2mm, F.Cu at (114.5, 122.2)
- added U20: MIC2009A-1YM6-TR, Common:SOT-23-6_Handsoldering, F.Cu at (127.8, 126.0)
- added U21: INA226AIDGSR, Common:SOP50P490X110-10N, F.Cu at (126.4, 130.2)
- added X3: 32.768KHZ, Oscillator:Oscillator_SMD_ECS_2520MV-xxx-xx-4Pin_2.5x2.0mm, F.Cu at (105.2, 110.9)
- moved D5 52.6 mm to (72.8, 137.9), turned to 90 degrees
- moved D6 51.5 mm to (74.5, 137.9), turned to 90 degrees
- moved D7 50.5 mm to (76.1, 137.9), turned to 90 degrees
- moved D8 49.5 mm to (77.8, 137.9), turned to 90 degrees
- moved R45 49.2 mm to (72.8, 135.1), turned to -90 degrees
- moved D9 48.6 mm to (79.4, 137.9), turned to 90 degrees
- moved R46 48.0 mm to (74.4, 135.1), turned to -90 degrees
- moved R47 46.8 mm to (76.1, 135.1), turned to -90 degrees
- moved R48 45.8 mm to (77.8, 135.1), turned to -90 degrees
- moved R49 44.9 mm to (79.4, 135.1), turned to -90 degrees
- moved C55 1.86 mm to (98.8, 109.5), turned to 180 degrees
- moved X2 1.72 mm to (102.0, 110.7), turned to 0 degrees
- moved C39 1.53 mm to (102.3, 108.5)
- moved R38 1.17 mm to (92.4, 119.9)
- moved C57 0.39 mm to (92.5, 124.5)
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- renumbered C48 to C55, C49 to C56, C50 to C57, C51 to C58, C52 to C59, C53 to C60, C54 to C61, C55 to C62, C56 to C63, C57 to C64, C58 to C68, C59 to C69, R23 to R25, R24 to R26, R25 to R35, R26 to R38, R27 to R41, R28 to R42, R29 to R43, R30 to R44, R31 to R45, R32 to R46, R33 to R47, R34 to R48, R35 to R49, R36 to R50, U10 to U15, U11 to U18
Connections:
- net GND renamed /GND
- C11 pad 1: /INTERBOARD_CONNECTOR2/3V3_18_RF1_COMM -> /3V3_COMM
- C12 pad 2: /INTERBOARD_CONNECTOR2/3V3_18_RF1_COMM -> /3V3_COMM
- C15 pad 1: /INTERBOARD_CONNECTOR2/3V3_18_RF1_COMM -> /3V3_COMM
- C27 pad 1: /INTERBOARD_CONNECTOR2/3V3_18_RF1_COMM -> /3V3_COMM
- C29 pad 1: /INTERBOARD_CONNECTOR2/3V3_18_RF1_COMM -> /3V3_COMM
- C3 pad 1: /INTERBOARD_CONNECTOR2/3V3_18_RF1_COMM -> /3V3_COMM
- C37 pad 1: /INTERBOARD_CONNECTOR2/3V3_18_RF1_COMM -> /3V3_COMM
- C38 pad 1: /INTERBOARD_CONNECTOR2/3V3_18_RF1_COMM -> /3V3_COMM
- FB1 pad 1: /INTERBOARD_CONNECTOR2/3V3_18_RF1_COMM -> /3V3_COMM
- FB2 pad 2: /INTERBOARD_CONNECTOR2/3V3_18_RF1_COMM -> /3V3_COMM
- FB3 pad 2: /INTERBOARD_CONNECTOR2/3V3_18_RF1_COMM -> /3V3_COMM
- FB4 pad 2: /INTERBOARD_CONNECTOR2/3V3_18_RF1_COMM -> /3V3_COMM
- J1 pad 2: /INTERBOARD_CONNECTOR2/3V3_18_RF1_COMM -> /3V3_COMM
- J2 pad 6: /INTERBOARD_CONNECTOR2/3V3_18_RF1_COMM -> /3V3_COMM
- J3 pad 3: /INTERBOARD_CONNECTOR2/3V3_18_RF1_COMM -> /3V3_COMM
- J4 pad 3: /INTERBOARD_CONNECTOR2/3V3_18_RF1_COMM -> /3V3_COMM
- R1 pad 2: /INTERBOARD_CONNECTOR2/3V3_18_RF1_COMM -> /3V3_COMM
- R18 pad 1: /INTERBOARD_CONNECTOR2/3V3_18_RF1_COMM -> /3V3_COMM
- R19 pad 2: /INTERBOARD_CONNECTOR2/3V3_18_RF1_COMM -> /3V3_COMM
- R3 pad 2: /INTERBOARD_CONNECTOR2/3V3_18_RF1_COMM -> /3V3_COMM
- R9 pad 2: /INTERBOARD_CONNECTOR2/3V3_18_RF1_COMM -> /3V3_COMM
- U15 pad 2: unconnected-(U10-PC13-Pad2) -> /CAN Bridge/PMIC/HSE_EN
- U15 pad 26: unconnected-(U10-PB0-Pad26) -> /CAN Bridge/Power_INT
- U15 pad 29: unconnected-(U10-PB10-Pad29) -> /CAN Bridge/I2C2_SCL
- U15 pad 3: unconnected-(U10-PC14-Pad3) -> /CAN Bridge/PMIC/OSC32_IN
- U15 pad 30: unconnected-(U10-PB11-Pad30) -> /CAN Bridge/I2C2_SDA
- U15 pad 37: unconnected-(U10-PC6-Pad37) -> /CAN Bridge/PMIC/LED1
- U15 pad 38: unconnected-(U10-PC7-Pad38) -> /CAN Bridge/PMIC/LED2
- U15 pad 39: unconnected-(U10-PC8-Pad39) -> /CAN Bridge/PMIC/LED3
- U15 pad 40: unconnected-(U10-PC9-Pad40) -> /CAN Bridge/PMIC/LED4
- U15 pad 41: unconnected-(U10-PA8-Pad41) -> /CAN Bridge/PMIC/LED5
- U15 pad 51: /CAN Bridge/PMIC/LED1 -> Net-(U15-PC10)
- U15 pad 52: /CAN Bridge/PMIC/LED2 -> /CAN Bridge/MRAM/SPI_MISO
- U15 pad 53: /CAN Bridge/PMIC/LED3 -> Net-(U15-PC12)
- U15 pad 54: unconnected-(U10-PD2-Pad54) -> /CAN Bridge/MRAM/SPI_CS
- U15 pad 55: /CAN Bridge/PMIC/LED4 -> /CAN Bridge/Power_RST
- U15 pad 56: /CAN Bridge/PMIC/LED5 -> unconnected-(U15-PB4-Pad56)
- U2 pad 3: /INTERBOARD_CONNECTOR2/3V3_18_RF1_COMM -> /3V3_COMM
- U7 pad 23: /INTERBOARD_CONNECTOR2/3V3_18_RF1_COMM -> /3V3_COMM
- X1 pad 4: /INTERBOARD_CONNECTOR2/3V3_18_RF1_COMM -> /3V3_COMM
- X2 pad 1: /INTERBOARD_CONNECTOR2/3V3_17_RF1_BRIDGE -> /CAN Bridge/PMIC/HSE_EN
Routing:
- net /CAN Bridge/I2C2_SCL: track 0.00 -> 108.0 mm, vias 0 -> 2
- net /CAN Bridge/I2C2_SDA: track 0.00 -> 106.9 mm, vias 0 -> 2
- net /3V3_COMM: track 0.00 -> 84.6 mm, vias 0 -> 14
- net /INTERBOARD_CONNECTOR2/3V3_18_RF1_COMM: track 57.3 -> 96.4 mm, vias 13 -> 7
- net /CAN Bridge/3V3_MRAM: track 0.00 -> 30.0 mm, vias 0 -> 4
- net /GND: track 217.7 -> 247.3 mm, vias 181 -> 207
- net /CAN Bridge/Power_INT: track 0.00 -> 28.2 mm, vias 0 -> 2
- net /CAN Bridge/Power Switch/INT3: track 0.00 -> 28.2 mm, vias 0 -> 2
- net /CAN Bridge/Power Switch/INT2: track 0.00 -> 26.2 mm
- net /CAN Bridge/Power_RST: track 0.00 -> 24.7 mm
- net /CAN Bridge/Power Switch/INT1: track 0.00 -> 24.2 mm, vias 0 -> 2
- net /CAN Bridge/Power Switch/INT0: track 0.00 -> 18.9 mm, vias 0 -> 2
- net /CAN Bridge/Power Switch/ENABLE2: track 0.00 -> 17.5 mm, vias 0 -> 2
- net /CAN Bridge/PMIC/HSE_EN: track 0.00 -> 17.3 mm
- net /CAN Bridge/Power Switch/ENABLE3: track 0.00 -> 16.9 mm
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- added copper zone on In2.Cu, net /3V3_COMM
- added copper zone on In2.Cu, net /CAN Bridge/3V3_MRAM
